File: Hardware/PCB/Mk1/Rev1/KBUltraMk1/KBUltraMk1.kicad_pcb (KiCad board)
At the start: 2 copper layers, 310 x 125 mm, 344 parts, among them SW1 SW_SPST, SW10 SW_SPST, SW11 SW_SPST, SW12 SW_SPST, SW13 SW_SPST, SW14 SW_SPST, SW15 SW_SPST, SW16 SW_SPST, SW17 SW_SPST, SW18 SW_SPST, SW19 SW_SPST, SW2 SW_SPST, SW20 SW_SPST, SW21 SW_SPST, SW22 SW_SPST, SW23 SW_SPST, SW24 SW_SPST, SW25 SW_SPST, SW26 SW_SPST, SW27 SW_SPST, SW28 SW_SPST, SW29 SW_SPST, SW3 SW_SPST, SW30 SW_SPST, SW31 SW_SPST, SW32 SW_SPST, SW33 SW_SPST, SW34 SW_SPST, SW35 SW_SPST, SW36 SW_SPST, SW37 SW_SPST, SW38 SW_SPST, SW39 SW_SPST, SW4 SW_SPST, SW40 SW_SPST, SW41 SW_SPST, SW42 SW_SPST, SW43 SW_SPST, SW44 SW_SPST, SW45 SW_SPST, SW46 SW_SPST, SW47 SW_SPST, SW48 SW_SPST, SW49 SW_SPST, SW5 SW_SPST, SW50 SW_SPST, SW51 SW_SPST, SW52 SW_SPST, SW53 SW_SPST, SW54 SW_SPST, SW55 SW_SPST, SW56 SW_SPST, SW57 SW_SPST, SW58 SW_SPST, SW59 SW_SPST, SW6 SW_SPST, SW60 SW_SPST, SW61 SW_SPST, SW62 SW_SPST, SW63 SW_SPST, SW64 SW_SPST, SW65 SW_SPST, SW66 SW_SPST, SW67 SW_SPST, SW68 SW_SPST, SW69 SW_SPST, SW7 SW_SPST, SW70 SW_SPST, SW71 SW_SPST, SW72 SW_SPST, SW73 SW_SPST, SW74 SW_SPST, SW75 SW_SPST, SW8 SW_SPST, SW9 SW_SPST

Commit message: Added RP MCU
Parts:
- removed C301, C302, C303, C304, C305, C306, C307, C308, C309, C310, C311, C312, C313, C314, C315, C316, C317, C318, C319, C320, C321, C322, C323, C324, C325, C326, C327, C328, C329, C330, C331, C332, C333, C334, C335, C336, C337, C338, C339, C340, C341, C342, C343, C344, C345, C346, C347, C348, C349, C350, C351, C352, C353, C354, C355, C356, C357, C358, C359, C360, C361, C362, C363, C364, C365, C366, C367, C368, C369, C370, C371, C372, C373, C374, C375, C376, C377, C378, C379, C380, C381, C382, C383, C384, C385, C386, C387, C388, C389, C390: 100n, Capacitor_SMD:C_0603_1608Metric
- removed D1, D10, D11, D12, D13, D14, D15, D16, D17, D18, D19, D2, D20, D21, D22, D23, D24, D25, D26, D27, D28, D29, D3, D30, D31, D32, D33, D34, D35, D36, D37, D38, D39, D4, D40, D41, D42, D43, D44, D45, D46, D47, D48, D49, D5, D50, D51, D52, D53, D54, D55, D56, D57, D58, D59, D6, D60, D61, D62, D63, D64, D65, D66, D67, D68, D69, D7, D70, D71, D72, D73, D74, D75, D8, D9: D, Diode_SMD:D_SOD-123
- removed D301, D302, D303, D304, D305, D306, D307, D308, D309, D310, D311, D312, D313, D314, D315, D316, D317, D318, D319, D320, D321, D322, D323, D324, D325, D326, D327, D328, D329, D330, D331, D332, D333, D334, D335, D336, D337, D338, D339, D340, D341, D342, D343, D344, D345, D346, D347, D348, D349, D350, D351, D352, D353, D354, D355, D356, D357, D358, D359, D360, D361, D362, D363, D364, D365, D366, D367, D368, D369, D370, D371, D372, D373, D374, D375, D376, D377, D378, D379, D380, D381, D382, D383, D384, D385, D386, D387, D388, D389, D390: SK6812MINI-E, LED_SMD:LED_SK6812MINI-E_3.2x2.8mm_P1.5mm_ReverseMount
- removed H1, H2, H3, H4: Stabalizer 2.00u, PCM_Mounting_Keyboard_Stabilizer:Stabilizer_Cherry_MX_2.00u
- removed H10, H11, H12, H13, H6, H7, H8, H9: MountingHole_Pad, MountingHole:MountingHole_3.2mm_M3_Pad_Via
- removed H5: Stabalizer 6.25u, PCM_Mounting_Keyboard_Stabilizer:Stabilizer_Cherry_MX_6.25u
- removed R301: 500R, Resistor_SMD:R_0603_1608Metric
- removed SW1, SW10, SW11, SW12, SW13, SW14, SW15, SW16, SW17, SW18, SW19, SW2, SW20, SW21, SW22, SW23, SW24, SW26, SW28, SW29, SW3, SW30, SW31, SW32, SW33, SW34, SW35, SW36, SW37, SW38, SW39, SW4, SW41, SW43, SW44, SW45, SW46, SW47, SW48, SW49, SW5, SW50, SW51, SW52, SW53, SW55, SW57, SW58, SW59, SW6, SW60, SW61, SW62, SW63, SW64, SW65, SW66, SW7, SW8, SW9: SW_SPST, PCM_Switch_Keyboard_Hotswap_Kailh:SW_Hotswap_Kailh_MX_Plated_1.00u
- removed SW25: SW_SPST, PCM_Switch_Keyboard_Hotswap_Kailh:SW_Hotswap_Kailh_MX_Plated_2.00u
- removed SW27, SW40: SW_SPST, PCM_Switch_Keyboard_Hotswap_Kailh:SW_Hotswap_Kailh_MX_Plated_1.50u
- removed SW42: SW_SPST, PCM_Switch_Keyboard_Hotswap_Kailh:SW_Hotswap_Kailh_MX_Plated_1.75u
- removed SW54, SW56: SW_SPST, PCM_Switch_Keyboard_Hotswap_Kailh:SW_Hotswap_Kailh_MX_Plated_2.25u
- removed SW67: SW_SPST, PCM_Switch_Keyboard_Hotswap_Kailh:SW_Hotswap_Kailh_MX_Plated_2.75u
- removed SW68, SW69, SW70, SW72, SW73, SW74, SW75: SW_SPST, PCM_Switch_Keyboard_Hotswap_Kailh:SW_Hotswap_Kailh_MX_Plated_1.25u
- removed SW71: SW_SPST, PCM_Switch_Keyboard_Hotswap_Kailh:SW_Hotswap_Kailh_MX_Plated_6.25u
- added C101: 4u7, Capacitor_SMD:C_0603_1608Metric, F.Cu at (158.0, 208.1)
- added C102: 100n, Capacitor_SMD:C_0603_1608Metric, F.Cu at (158.0, 210.6)
- added C103: 100n, Capacitor_SMD:C_0603_1608Metric, F.Cu at (158.0, 213.1)
- added C104: 100n, Capacitor_SMD:C_0603_1608Metric, F.Cu at (158.0, 215.6)
- added C105: 100n, Capacitor_SMD:C_0603_1608Metric, F.Cu at (158.0, 218.1)
- added C106: 100n, Capacitor_SMD:C_0603_1608Metric, F.Cu at (158.0, 220.7)
- added C107: 100n, Capacitor_SMD:C_0603_1608Metric, F.Cu at (158.0, 223.2)
- added C108: 100n, Capacitor_SMD:C_0603_1608Metric, F.Cu at (162.0, 208.1)
- added C109: 100n, Capacitor_SMD:C_0603_1608Metric, F.Cu at (162.0, 210.6)
- added C110: 4u7, Capacitor_SMD:C_0603_1608Metric, F.Cu at (162.0, 213.1)
- added C111: 4u7, Capacitor_SMD:C_0603_1608Metric, F.Cu at (162.0, 215.6)
- added C112: 4u7, Capacitor_SMD:C_0603_1608Metric, F.Cu at (162.0, 218.1)
- added C113: 4u7, Capacitor_SMD:C_0603_1608Metric, F.Cu at (162.0, 220.7)
- added C114: 100n, Capacitor_SMD:C_0603_1608Metric, F.Cu at (162.0, 223.2)
- added C115: 100n, Capacitor_SMD:C_0603_1608Metric, F.Cu at (166.0, 208.1)
- added C116: 100n, Capacitor_SMD:C_0603_1608Metric, F.Cu at (166.0, 210.6)
- added C117: 100n, Capacitor_SMD:C_0603_1608Metric, F.Cu at (166.0, 213.1)
- added C118: 100n, Capacitor_SMD:C_0603_1608Metric, F.Cu at (166.0, 215.6)
- added C201: 100n, Capacitor_SMD:C_0603_1608Metric, B.Cu at (74.2, 82.3)
- added C202: 100n, Capacitor_SMD:C_0603_1608Metric, B.Cu at (131.4, 82.3)
- added C203: 100n, Capacitor_SMD:C_0603_1608Metric, B.Cu at (150.4, 82.3)
- added C204: 100n, Capacitor_SMD:C_0603_1608Metric, B.Cu at (169.5, 82.3)
- added C205: 100n, Capacitor_SMD:C_0603_1608Metric, B.Cu at (188.5, 82.3)
- added C206: 100n, Capacitor_SMD:C_0603_1608Metric, B.Cu at (207.6, 82.3)
- added C207: 100n, Capacitor_SMD:C_0603_1608Metric, B.Cu at (226.6, 82.3)
- added C208: 100n, Capacitor_SMD:C_0603_1608Metric, B.Cu at (245.7, 82.3)
- added C209: 100n, Capacitor_SMD:C_0603_1608Metric, B.Cu at (264.7, 82.3)
- added C210: 100n, Capacitor_SMD:C_0603_1608Metric, B.Cu at (283.8, 82.3)
- added C211: 100n, Capacitor_SMD:C_0603_1608Metric, B.Cu at (74.2, 101.3)
- added C212: 100n, Capacitor_SMD:C_0603_1608Metric, B.Cu at (93.3, 101.3)
- added C213: 100n, Capacitor_SMD:C_0603_1608Metric, B.Cu at (112.3, 101.3)
- added C214: 100n, Capacitor_SMD:C_0603_1608Metric, B.Cu at (131.4, 101.3)
- added C215: 100n, Capacitor_SMD:C_0603_1608Metric, B.Cu at (150.4, 101.3)
- added C216: 100n, Capacitor_SMD:C_0603_1608Metric, B.Cu at (169.5, 101.3)
- added C217: 100n, Capacitor_SMD:C_0603_1608Metric, B.Cu at (188.5, 101.3)
- added C218: 100n, Capacitor_SMD:C_0603_1608Metric, B.Cu at (207.6, 101.3)
- added C219: 100n, Capacitor_SMD:C_0603_1608Metric, B.Cu at (226.6, 101.3)
- added C220: 100n, Capacitor_SMD:C_0603_1608Metric, B.Cu at (245.7, 101.3)
- added C221: 100n, Capacitor_SMD:C_0603_1608Metric, B.Cu at (264.7, 101.3)
- added C222: 100n, Capacitor_SMD:C_0603_1608Metric, B.Cu at (283.8, 101.3)
- added C223: 100n, Capacitor_SMD:C_0603_1608Metric, B.Cu at (302.8, 101.3)
- added C224: 100n, Capacitor_SMD:C_0603_1608Metric, B.Cu at (321.9, 101.3)
- added C225: 100n, Capacitor_SMD:C_0603_1608Metric, B.Cu at (350.5, 101.3)
- added C226: 100n, Capacitor_SMD:C_0603_1608Metric, B.Cu at (74.2, 120.4)
- added C227: 100n, Capacitor_SMD:C_0603_1608Metric, B.Cu at (98.1, 120.4)
- added C228: 100n, Capacitor_SMD:C_0603_1608Metric, B.Cu at (121.9, 120.4)
- added C229: 100n, Capacitor_SMD:C_0603_1608Metric, B.Cu at (140.9, 120.4)
- added C230: 100n, Capacitor_SMD:C_0603_1608Metric, B.Cu at (160.0, 120.4)
- added C231: 100n, Capacitor_SMD:C_0603_1608Metric, B.Cu at (179.0, 120.4)
- added C232: 100n, Capacitor_SMD:C_0603_1608Metric, B.Cu at (198.1, 120.4)
- added C233: 100n, Capacitor_SMD:C_0603_1608Metric, B.Cu at (217.1, 120.4)
- added C234: 100n, Capacitor_SMD:C_0603_1608Metric, B.Cu at (236.2, 120.4)
- added C235: 100n, Capacitor_SMD:C_0603_1608Metric, B.Cu at (255.2, 120.4)
- added C236: 100n, Capacitor_SMD:C_0603_1608Metric, B.Cu at (274.3, 120.4)
- added C237: 100n, Capacitor_SMD:C_0603_1608Metric, B.Cu at (293.3, 120.4)
- added C238: 100n, Capacitor_SMD:C_0603_1608Metric, B.Cu at (312.4, 120.4)
- added C239: 100n, Capacitor_SMD:C_0603_1608Metric, B.Cu at (331.4, 120.4)
- added C240: 100n, Capacitor_SMD:C_0603_1608Metric, B.Cu at (355.2, 120.4)
- added C241: 100n, Capacitor_SMD:C_0603_1608Metric, B.Cu at (74.2, 139.4)
- added C242: 100n, Capacitor_SMD:C_0603_1608Metric, B.Cu at (100.4, 139.4)
- added C243: 100n, Capacitor_SMD:C_0603_1608Metric, B.Cu at (126.6, 139.4)
- added C244: 100n, Capacitor_SMD:C_0603_1608Metric, B.Cu at (145.7, 139.4)
- added C245: 100n, Capacitor_SMD:C_0603_1608Metric, B.Cu at (164.7, 139.4)
- added C246: 100n, Capacitor_SMD:C_0603_1608Metric, B.Cu at (183.8, 139.4)
- added C247: 100n, Capacitor_SMD:C_0603_1608Metric, B.Cu at (202.8, 139.4)
- added C248: 100n, Capacitor_SMD:C_0603_1608Metric, B.Cu at (221.9, 139.4)
- added C249: 100n, Capacitor_SMD:C_0603_1608Metric, B.Cu at (240.9, 139.4)
- added C250: 100n, Capacitor_SMD:C_0603_1608Metric, B.Cu at (260.0, 139.4)
- added C251: 100n, Capacitor_SMD:C_0603_1608Metric, B.Cu at (279.0, 139.4)
- added C252: 100n, Capacitor_SMD:C_0603_1608Metric, B.Cu at (298.1, 139.4)
- added C253: 100n, Capacitor_SMD:C_0603_1608Metric, B.Cu at (317.1, 139.4)
- added C254: 100n, Capacitor_SMD:C_0603_1608Metric, B.Cu at (348.1, 139.4)
- added C255: 100n, Capacitor_SMD:C_0603_1608Metric, B.Cu at (74.2, 158.5)
- added C256: 100n, Capacitor_SMD:C_0603_1608Metric, B.Cu at (105.2, 158.5)
- added C257: 100n, Capacitor_SMD:C_0603_1608Metric, B.Cu at (136.2, 158.5)
- added C258: 100n, Capacitor_SMD:C_0603_1608Metric, B.Cu at (155.2, 158.5)
- added C259: 100n, Capacitor_SMD:C_0603_1608Metric, B.Cu at (174.3, 158.5)
- added C260: 100n, Capacitor_SMD:C_0603_1608Metric, B.Cu at (193.3, 158.5)
- added C261: 100n, Capacitor_SMD:C_0603_1608Metric, B.Cu at (212.4, 158.5)
- added C262: 100n, Capacitor_SMD:C_0603_1608Metric, B.Cu at (231.4, 158.5)
- added C263: 100n, Capacitor_SMD:C_0603_1608Metric, B.Cu at (250.5, 158.5)
- added C264: 100n, Capacitor_SMD:C_0603_1608Metric, B.Cu at (269.5, 158.5)
- added C265: 100n, Capacitor_SMD:C_0603_1608Metric, B.Cu at (288.6, 158.5)
- added C266: 100n, Capacitor_SMD:C_0603_1608Metric, B.Cu at (307.6, 158.5)
- added C267: 100n, Capacitor_SMD:C_0603_1608Metric, B.Cu at (343.3, 158.5)
- added C268: 100n, Capacitor_SMD:C_0603_1608Metric, B.Cu at (95.7, 177.5)
- added C269: 100n, Capacitor_SMD:C_0603_1608Metric, B.Cu at (119.5, 177.5)
- added C270: 100n, Capacitor_SMD:C_0603_1608Metric, B.Cu at (143.3, 177.5)
- added C271: 100n, Capacitor_SMD:C_0603_1608Metric, B.Cu at (214.7, 177.5)
- added C272: 100n, Capacitor_SMD:C_0603_1608Metric, B.Cu at (286.2, 177.5)
- added C273: 100n, Capacitor_SMD:C_0603_1608Metric, B.Cu at (310.0, 177.5)
- added C274: 100n, Capacitor_SMD:C_0603_1608Metric, B.Cu at (333.8, 177.5)
- added C275: 100n, Capacitor_SMD:C_0603_1608Metric, B.Cu at (357.6, 177.5)
- added C276: 100n, Capacitor_SMD:C_0603_1608Metric, F.Cu at (-72.8, 237.8)
- added C277: 100n, Capacitor_SMD:C_0603_1608Metric, F.Cu at (-72.8, 240.3)
- added C278: 100n, Capacitor_SMD:C_0603_1608Metric, F.Cu at (-72.8, 242.8)
- added C279: 100n, Capacitor_SMD:C_0603_1608Metric, F.Cu at (-72.8, 245.3)
- added C280: 100n, Capacitor_SMD:C_0603_1608Metric, F.Cu at (-72.8, 247.8)
- added C281: 100n, Capacitor_SMD:C_0603_1608Metric, F.Cu at (-72.8, 250.3)
- added C282: 100n, Capacitor_SMD:C_0603_1608Metric, F.Cu at (-72.8, 252.8)
- added C283: 100n, Capacitor_SMD:C_0603_1608Metric, F.Cu at (-72.8, 255.3)
- added C284: 100n, Capacitor_SMD:C_0603_1608Metric, F.Cu at (-72.8, 257.9)
- added C285: 100n, Capacitor_SMD:C_0603_1608Metric, B.Cu at (193.3, 177.6)
- added C286: 100n, Capacitor_SMD:C_0603_1608Metric, B.Cu at (231.4, 177.6)
- added C287: 100n, Capacitor_SMD:C_0603_1608Metric, F.Cu at (-68.8, 230.2)
- added C288: 100n, Capacitor_SMD:C_0603_1608Metric, F.Cu at (-68.8, 232.8)
- added C289: 100n, Capacitor_SMD:C_0603_1608Metric, F.Cu at (-68.8, 235.3)
- added C290: 100n, Capacitor_SMD:C_0603_1608Metric, F.Cu at (-68.8, 237.8)
- added D201: D, Diode_SMD:D_SOD-123, B.Cu at (79.3, 78.7)
- added D202: D, Diode_SMD:D_SOD-123, B.Cu at (136.5, 78.7)
- added D203: D, Diode_SMD:D_SOD-123, B.Cu at (155.5, 78.7)
- added D204: D, Diode_SMD:D_SOD-123, B.Cu at (174.6, 78.7)
- added D205: D, Diode_SMD:D_SOD-123, B.Cu at (193.6, 78.7)
- added D206: D, Diode_SMD:D_SOD-123, B.Cu at (212.7, 78.7)
- added D207: D, Diode_SMD:D_SOD-123, B.Cu at (231.7, 78.7)
- added D208: D, Diode_SMD:D_SOD-123, B.Cu at (250.8, 78.7)
- added D209: D, Diode_SMD:D_SOD-123, B.Cu at (269.8, 78.7)
- added D210: D, Diode_SMD:D_SOD-123, B.Cu at (288.9, 78.7)
- added D211: D, Diode_SMD:D_SOD-123, B.Cu at (79.3, 97.7)
- added D212: D, Diode_SMD:D_SOD-123, B.Cu at (98.4, 97.7)
- added D213: D, Diode_SMD:D_SOD-123, B.Cu at (117.4, 97.7)
- added D214: D, Diode_SMD:D_SOD-123, B.Cu at (136.5, 97.7)
- added D215: D, Diode_SMD:D_SOD-123, B.Cu at (155.5, 97.7)
- added D216: D, Diode_SMD:D_SOD-123, B.Cu at (174.6, 97.7)
- added D217: D, Diode_SMD:D_SOD-123, B.Cu at (193.6, 97.7)
- added D218: D, Diode_SMD:D_SOD-123, B.Cu at (212.7, 97.7)
- added D219: D, Diode_SMD:D_SOD-123, B.Cu at (231.7, 97.7)
- added D220: D, Diode_SMD:D_SOD-123, B.Cu at (250.8, 97.7)
- added D221: D, Diode_SMD:D_SOD-123, B.Cu at (269.8, 97.7)
- added D222: D, Diode_SMD:D_SOD-123, B.Cu at (288.9, 97.7)
- added D223: D, Diode_SMD:D_SOD-123, B.Cu at (307.9, 97.7)
- added D224: D, Diode_SMD:D_SOD-123, B.Cu at (327.0, 97.7)
- added D225: D, Diode_SMD:D_SOD-123, B.Cu at (355.5, 97.7)
- added D226: D, Diode_SMD:D_SOD-123, B.Cu at (79.3, 116.8)
- added D227: D, Diode_SMD:D_SOD-123, B.Cu at (103.1, 116.8)
- added D228: D, Diode_SMD:D_SOD-123, B.Cu at (126.9, 116.8)
- added D229: D, Diode_SMD:D_SOD-123, B.Cu at (146.0, 116.8)
- added D230: D, Diode_SMD:D_SOD-123, B.Cu at (165.0, 116.8)
- added D231: D, Diode_SMD:D_SOD-123, B.Cu at (184.1, 116.8)
- added D232: D, Diode_SMD:D_SOD-123, B.Cu at (203.1, 116.8)
- added D233: D, Diode_SMD:D_SOD-123, B.Cu at (222.2, 116.8)
- added D234: D, Diode_SMD:D_SOD-123, B.Cu at (241.2, 116.8)
- added D235: D, Diode_SMD:D_SOD-123, B.Cu at (260.3, 116.8)
- added D236: D, Diode_SMD:D_SOD-123, B.Cu at (279.3, 116.8)
- added D237: D, Diode_SMD:D_SOD-123, B.Cu at (298.4, 116.8)
- added D238: D, Diode_SMD:D_SOD-123, B.Cu at (317.4, 116.8)
- added D239: D, Diode_SMD:D_SOD-123, B.Cu at (336.5, 116.8)
- added D240: D, Diode_SMD:D_SOD-123, B.Cu at (360.3, 116.8)
- added D241: D, Diode_SMD:D_SOD-123, B.Cu at (79.3, 135.8)
- added D242: D, Diode_SMD:D_SOD-123, B.Cu at (105.5, 135.8)
- added D243: D, Diode_SMD:D_SOD-123, B.Cu at (131.7, 135.8)
- added D244: D, Diode_SMD:D_SOD-123, B.Cu at (150.8, 135.8)
- added D245: D, Diode_SMD:D_SOD-123, B.Cu at (169.8, 135.8)
- added D246: D, Diode_SMD:D_SOD-123, B.Cu at (188.9, 135.8)
- added D247: D, Diode_SMD:D_SOD-123, B.Cu at (207.9, 135.8)
- added D248: D, Diode_SMD:D_SOD-123, B.Cu at (227.0, 135.8)
- added D249: D, Diode_SMD:D_SOD-123, B.Cu at (246.0, 135.8)
- added D250: D, Diode_SMD:D_SOD-123, B.Cu at (265.1, 135.8)
- added D251: D, Diode_SMD:D_SOD-123, B.Cu at (284.1, 135.8)
- added D252: D, Diode_SMD:D_SOD-123, B.Cu at (303.2, 135.8)
- added D253: D, Diode_SMD:D_SOD-123, B.Cu at (322.2, 135.8)
- added D254: D, Diode_SMD:D_SOD-123, B.Cu at (353.2, 135.8)
- added D255: D, Diode_SMD:D_SOD-123, B.Cu at (79.3, 154.9)
- added D256: D, Diode_SMD:D_SOD-123, B.Cu at (110.3, 154.9)
- added D257: D, Diode_SMD:D_SOD-123, B.Cu at (141.2, 154.9)
- added D258: D, Diode_SMD:D_SOD-123, B.Cu at (160.3, 154.9)
- added D259: D, Diode_SMD:D_SOD-123, B.Cu at (179.3, 154.9)
- added D260: D, Diode_SMD:D_SOD-123, B.Cu at (198.4, 154.9)
- added D261: D, Diode_SMD:D_SOD-123, B.Cu at (217.4, 154.9)
- added D262: D, Diode_SMD:D_SOD-123, B.Cu at (236.5, 154.9)
- added D263: D, Diode_SMD:D_SOD-123, B.Cu at (255.5, 154.9)
- added D264: D, Diode_SMD:D_SOD-123, B.Cu at (274.6, 154.9)
- added D265: D, Diode_SMD:D_SOD-123, B.Cu at (293.6, 154.9)
- added D266: D, Diode_SMD:D_SOD-123, B.Cu at (312.7, 154.9)
- added D267: D, Diode_SMD:D_SOD-123, B.Cu at (348.4, 154.9)
- added D268: D, Diode_SMD:D_SOD-123, B.Cu at (100.8, 173.9)
- added D269: D, Diode_SMD:D_SOD-123, B.Cu at (124.6, 173.9)
- added D270: D, Diode_SMD:D_SOD-123, B.Cu at (148.4, 173.9)
- added D271: D, Diode_SMD:D_SOD-123, B.Cu at (219.8, 173.9)
- added D272: D, Diode_SMD:D_SOD-123, B.Cu at (291.3, 173.9)
- added D273: D, Diode_SMD:D_SOD-123, B.Cu at (315.1, 173.9)
- added D274: D, Diode_SMD:D_SOD-123, B.Cu at (338.9, 173.9)
- added D275: D, Diode_SMD:D_SOD-123, B.Cu at (362.7, 173.9)
- added H201: Stabalizer 2.00u, PCM_Mounting_Keyboard_Stabilizer:Stabilizer_Cherry_MX_2.00u, F.Cu at (105.2, 150.9)
- added H202: MountingHole_Pad, MountingHole:MountingHole_3.2mm_M3_Pad_Via, F.Cu at (297.6, 74.7)
- added H203: Stabalizer 2.00u, PCM_Mounting_Keyboard_Stabilizer:Stabilizer_Cherry_MX_2.00u, F.Cu at (343.3, 150.9)
- added H204: MountingHole_Pad, MountingHole:MountingHole_3.2mm_M3_Pad_Via, F.Cu at (117.7, 74.7)
- added H205: Stabalizer 2.00u, PCM_Mounting_Keyboard_Stabilizer:Stabilizer_Cherry_MX_2.00u, F.Cu at (348.1, 131.8)
- added H206: MountingHole_Pad, MountingHole:MountingHole_3.2mm_M3_Pad_Via, F.Cu at (321.4, 150.5)
- added H207: Stabalizer 2.00u, PCM_Mounting_Keyboard_Stabilizer:Stabilizer_Cherry_MX_2.00u, F.Cu at (350.5, 93.7)
- added H208: MountingHole_Pad, MountingHole:MountingHole_3.2mm_M3_Pad_Via, F.Cu at (124.3, 150.9)
- added H209: Stabalizer 6.25u, PCM_Mounting_Keyboard_Stabilizer:Stabilizer_Cherry_MX_6.25u, F.Cu at (214.7, 169.9)
- added H210: MountingHole_Pad, MountingHole:MountingHole_3.2mm_M3_Pad_Via, F.Cu at (66.4, 64.1)
- added H211: MountingHole_Pad, MountingHole:MountingHole_3.2mm_M3_Pad_Via, F.Cu at (66.4, 180.5)
- added H212: MountingHole_Pad, MountingHole:MountingHole_3.2mm_M3_Pad_Via, F.Cu at (367.8, 180.5)
- added H213: MountingHole_Pad, MountingHole:MountingHole_3.2mm_M3_Pad_Via, F.Cu at (367.8, 64.1)
- added LED201: SK6812MINI-E, LED_SMD:LED_SK6812MINI-E_3.2x2.8mm_P1.5mm_ReverseMount, B.Cu at (74.2, 79.5)
- added LED202: SK6812MINI-E, LED_SMD:LED_SK6812MINI-E_3.2x2.8mm_P1.5mm_ReverseMount, B.Cu at (131.4, 79.5)
- added LED203: SK6812MINI-E, LED_SMD:LED_SK6812MINI-E_3.2x2.8mm_P1.5mm_ReverseMount, B.Cu at (150.4, 79.5)
- added LED204: SK6812MINI-E, LED_SMD:LED_SK6812MINI-E_3.2x2.8mm_P1.5mm_ReverseMount, B.Cu at (169.5, 79.5)
- added LED205: SK6812MINI-E, LED_SMD:LED_SK6812MINI-E_3.2x2.8mm_P1.5mm_ReverseMount, B.Cu at (188.5, 79.5)
- added LED206: SK6812MINI-E, LED_SMD:LED_SK6812MINI-E_3.2x2.8mm_P1.5mm_ReverseMount, B.Cu at (207.6, 79.5)
- added LED207: SK6812MINI-E, LED_SMD:LED_SK6812MINI-E_3.2x2.8mm_P1.5mm_ReverseMount, B.Cu at (226.6, 79.5)
- added LED208: SK6812MINI-E, LED_SMD:LED_SK6812MINI-E_3.2x2.8mm_P1.5mm_ReverseMount, B.Cu at (245.7, 79.5)
- added LED209: SK6812MINI-E, LED_SMD:LED_SK6812MINI-E_3.2x2.8mm_P1.5mm_ReverseMount, B.Cu at (264.7, 79.5)
- added LED210: SK6812MINI-E, LED_SMD:LED_SK6812MINI-E_3.2x2.8mm_P1.5mm_ReverseMount, B.Cu at (283.8, 79.5)
- added LED211: SK6812MINI-E, LED_SMD:LED_SK6812MINI-E_3.2x2.8mm_P1.5mm_ReverseMount, B.Cu at (74.2, 98.5)
- added LED212: SK6812MINI-E, LED_SMD:LED_SK6812MINI-E_3.2x2.8mm_P1.5mm_ReverseMount, B.Cu at (93.3, 98.5)
- added LED213: SK6812MINI-E, LED_SMD:LED_SK6812MINI-E_3.2x2.8mm_P1.5mm_ReverseMount, B.Cu at (112.3, 98.5)
- added LED214: SK6812MINI-E, LED_SMD:LED_SK6812MINI-E_3.2x2.8mm_P1.5mm_ReverseMount, B.Cu at (131.4, 98.5)
- added LED215: SK6812MINI-E, LED_SMD:LED_SK6812MINI-E_3.2x2.8mm_P1.5mm_ReverseMount, B.Cu at (150.4, 98.5)
- added LED216: SK6812MINI-E, LED_SMD:LED_SK6812MINI-E_3.2x2.8mm_P1.5mm_ReverseMount, B.Cu at (169.5, 98.5)
- added LED217: SK6812MINI-E, LED_SMD:LED_SK6812MINI-E_3.2x2.8mm_P1.5mm_ReverseMount, B.Cu at (188.5, 98.5)
- added LED218: SK6812MINI-E, LED_SMD:LED_SK6812MINI-E_3.2x2.8mm_P1.5mm_ReverseMount, B.Cu at (207.6, 98.5)
- added LED219: SK6812MINI-E, LED_SMD:LED_SK6812MINI-E_3.2x2.8mm_P1.5mm_ReverseMount, B.Cu at (226.6, 98.5)
- added LED220: SK6812MINI-E, LED_SMD:LED_SK6812MINI-E_3.2x2.8mm_P1.5mm_ReverseMount, B.Cu at (245.7, 98.5)
- added LED221: SK6812MINI-E, LED_SMD:LED_SK6812MINI-E_3.2x2.8mm_P1.5mm_ReverseMount, B.Cu at (264.7, 98.5)
- added LED222: SK6812MINI-E, LED_SMD:LED_SK6812MINI-E_3.2x2.8mm_P1.5mm_ReverseMount, B.Cu at (283.8, 98.5)
- added LED223: SK6812MINI-E, LED_SMD:LED_SK6812MINI-E_3.2x2.8mm_P1.5mm_ReverseMount, B.Cu at (302.8, 98.5)
- added LED224: SK6812MINI-E, LED_SMD:LED_SK6812MINI-E_3.2x2.8mm_P1.5mm_ReverseMount, B.Cu at (321.9, 98.5)
- added LED225: SK6812MINI-E, LED_SMD:LED_SK6812MINI-E_3.2x2.8mm_P1.5mm_ReverseMount, B.Cu at (350.5, 98.5)
- added LED226: SK6812MINI-E, LED_SMD:LED_SK6812MINI-E_3.2x2.8mm_P1.5mm_ReverseMount, B.Cu at (74.2, 117.6)
- added LED227: SK6812MINI-E, LED_SMD:LED_SK6812MINI-E_3.2x2.8mm_P1.5mm_ReverseMount, B.Cu at (98.1, 117.6)
- added LED228: SK6812MINI-E, LED_SMD:LED_SK6812MINI-E_3.2x2.8mm_P1.5mm_ReverseMount, B.Cu at (121.9, 117.6)
- added LED229: SK6812MINI-E, LED_SMD:LED_SK6812MINI-E_3.2x2.8mm_P1.5mm_ReverseMount, B.Cu at (140.9, 117.6)
- added LED230: SK6812MINI-E, LED_SMD:LED_SK6812MINI-E_3.2x2.8mm_P1.5mm_ReverseMount, B.Cu at (160.0, 117.6)
- added LED231: SK6812MINI-E, LED_SMD:LED_SK6812MINI-E_3.2x2.8mm_P1.5mm_ReverseMount, B.Cu at (179.0, 117.6)
- added LED232: SK6812MINI-E, LED_SMD:LED_SK6812MINI-E_3.2x2.8mm_P1.5mm_ReverseMount, B.Cu at (198.1, 117.6)
- added LED233: SK6812MINI-E, LED_SMD:LED_SK6812MINI-E_3.2x2.8mm_P1.5mm_ReverseMount, B.Cu at (217.1, 117.6)
- added LED234: SK6812MINI-E, LED_SMD:LED_SK6812MINI-E_3.2x2.8mm_P1.5mm_ReverseMount, B.Cu at (236.2, 117.6)
- added LED235: SK6812MINI-E, LED_SMD:LED_SK6812MINI-E_3.2x2.8mm_P1.5mm_ReverseMount, B.Cu at (255.2, 117.6)
- added LED236: SK6812MINI-E, LED_SMD:LED_SK6812MINI-E_3.2x2.8mm_P1.5mm_ReverseMount, B.Cu at (274.3, 117.6)
- added LED237: SK6812MINI-E, LED_SMD:LED_SK6812MINI-E_3.2x2.8mm_P1.5mm_ReverseMount, B.Cu at (293.3, 117.6)
- added LED238: SK6812MINI-E, LED_SMD:LED_SK6812MINI-E_3.2x2.8mm_P1.5mm_ReverseMount, B.Cu at (312.4, 117.6)
- added LED239: SK6812MINI-E, LED_SMD:LED_SK6812MINI-E_3.2x2.8mm_P1.5mm_ReverseMount, B.Cu at (331.4, 117.6)
- added LED240: SK6812MINI-E, LED_SMD:LED_SK6812MINI-E_3.2x2.8mm_P1.5mm_ReverseMount, B.Cu at (355.2, 117.6)
- added LED241: SK6812MINI-E, LED_SMD:LED_SK6812MINI-E_3.2x2.8mm_P1.5mm_ReverseMount, B.Cu at (74.2, 136.6)
- added LED242: SK6812MINI-E, LED_SMD:LED_SK6812MINI-E_3.2x2.8mm_P1.5mm_ReverseMount, B.Cu at (100.4, 136.6)
- added LED243: SK6812MINI-E, LED_SMD:LED_SK6812MINI-E_3.2x2.8mm_P1.5mm_ReverseMount, B.Cu at (126.6, 136.6)
- added LED244: SK6812MINI-E, LED_SMD:LED_SK6812MINI-E_3.2x2.8mm_P1.5mm_ReverseMount, B.Cu at (145.7, 136.6)
- added LED245: SK6812MINI-E, LED_SMD:LED_SK6812MINI-E_3.2x2.8mm_P1.5mm_ReverseMount, B.Cu at (164.7, 136.6)
- added LED246: SK6812MINI-E, LED_SMD:LED_SK6812MINI-E_3.2x2.8mm_P1.5mm_ReverseMount, B.Cu at (183.8, 136.6)
- added LED247: SK6812MINI-E, LED_SMD:LED_SK6812MINI-E_3.2x2.8mm_P1.5mm_ReverseMount, B.Cu at (202.8, 136.6)
- added LED248: SK6812MINI-E, LED_SMD:LED_SK6812MINI-E_3.2x2.8mm_P1.5mm_ReverseMount, B.Cu at (221.9, 136.6)
- added LED249: SK6812MINI-E, LED_SMD:LED_SK6812MINI-E_3.2x2.8mm_P1.5mm_ReverseMount, B.Cu at (240.9, 136.6)
- added LED250: SK6812MINI-E, LED_SMD:LED_SK6812MINI-E_3.2x2.8mm_P1.5mm_ReverseMount, B.Cu at (260.0, 136.6)
- added LED251: SK6812MINI-E, LED_SMD:LED_SK6812MINI-E_3.2x2.8mm_P1.5mm_ReverseMount, B.Cu at (279.0, 136.6)
- added LED252: SK6812MINI-E, LED_SMD:LED_SK6812MINI-E_3.2x2.8mm_P1.5mm_ReverseMount, B.Cu at (298.1, 136.6)
- added LED253: SK6812MINI-E, LED_SMD:LED_SK6812MINI-E_3.2x2.8mm_P1.5mm_ReverseMount, B.Cu at (317.1, 136.6)
- added LED254: SK6812MINI-E, LED_SMD:LED_SK6812MINI-E_3.2x2.8mm_P1.5mm_ReverseMount, B.Cu at (348.1, 136.6)
- added LED255: SK6812MINI-E, LED_SMD:LED_SK6812MINI-E_3.2x2.8mm_P1.5mm_ReverseMount, B.Cu at (74.2, 155.7)
- added LED256: SK6812MINI-E, LED_SMD:LED_SK6812MINI-E_3.2x2.8mm_P1.5mm_ReverseMount, B.Cu at (105.2, 155.7)
- added LED257: SK6812MINI-E, LED_SMD:LED_SK6812MINI-E_3.2x2.8mm_P1.5mm_ReverseMount, B.Cu at (136.2, 155.7)
- added LED258: SK6812MINI-E, LED_SMD:LED_SK6812MINI-E_3.2x2.8mm_P1.5mm_ReverseMount, B.Cu at (155.2, 155.7)
- added LED259: SK6812MINI-E, LED_SMD:LED_SK6812MINI-E_3.2x2.8mm_P1.5mm_ReverseMount, B.Cu at (174.3, 155.7)
- added LED260: SK6812MINI-E, LED_SMD:LED_SK6812MINI-E_3.2x2.8mm_P1.5mm_ReverseMount, B.Cu at (193.3, 155.7)
- added LED261: SK6812MINI-E, LED_SMD:LED_SK6812MINI-E_3.2x2.8mm_P1.5mm_ReverseMount, B.Cu at (212.4, 155.7)
- added LED262: SK6812MINI-E, LED_SMD:LED_SK6812MINI-E_3.2x2.8mm_P1.5mm_ReverseMount, B.Cu at (231.4, 155.7)
- added LED263: SK6812MINI-E, LED_SMD:LED_SK6812MINI-E_3.2x2.8mm_P1.5mm_ReverseMount, B.Cu at (250.5, 155.7)
- added LED264: SK6812MINI-E, LED_SMD:LED_SK6812MINI-E_3.2x2.8mm_P1.5mm_ReverseMount, B.Cu at (269.5, 155.7)
- added LED265: SK6812MINI-E, LED_SMD:LED_SK6812MINI-E_3.2x2.8mm_P1.5mm_ReverseMount, B.Cu at (288.6, 155.7)
- added LED266: SK6812MINI-E, LED_SMD:LED_SK6812MINI-E_3.2x2.8mm_P1.5mm_ReverseMount, B.Cu at (307.6, 155.7)
- added LED267: SK6812MINI-E, LED_SMD:LED_SK6812MINI-E_3.2x2.8mm_P1.5mm_ReverseMount, B.Cu at (343.3, 155.7)
- added LED268: SK6812MINI-E, LED_SMD:LED_SK6812MINI-E_3.2x2.8mm_P1.5mm_ReverseMount, B.Cu at (95.7, 174.7)
- added LED269: SK6812MINI-E, LED_SMD:LED_SK6812MINI-E_3.2x2.8mm_P1.5mm_ReverseMount, B.Cu at (119.5, 174.7)
- added LED270: SK6812MINI-E, LED_SMD:LED_SK6812MINI-E_3.2x2.8mm_P1.5mm_ReverseMount, B.Cu at (143.3, 174.7)
- added LED271: SK6812MINI-E, LED_SMD:LED_SK6812MINI-E_3.2x2.8mm_P1.5mm_ReverseMount, B.Cu at (214.7, 174.7)
- added LED272: SK6812MINI-E, LED_SMD:LED_SK6812MINI-E_3.2x2.8mm_P1.5mm_ReverseMount, B.Cu at (286.2, 174.7)
- added LED273: SK6812MINI-E, LED_SMD:LED_SK6812MINI-E_3.2x2.8mm_P1.5mm_ReverseMount, B.Cu at (310.0, 174.7)
- added LED274: SK6812MINI-E, LED_SMD:LED_SK6812MINI-E_3.2x2.8mm_P1.5mm_ReverseMount, B.Cu at (333.8, 174.7)
- added LED275: SK6812MINI-E, LED_SMD:LED_SK6812MINI-E_3.2x2.8mm_P1.5mm_ReverseMount, B.Cu at (357.6, 174.7)
- added LED276: SK6812MINI-E, LED_SMD:LED_SK6812MINI-E_3.2x2.8mm_P1.5mm_ReverseMount, F.Cu at (-34.5, 235.8)
- added LED277: SK6812MINI-E, LED_SMD:LED_SK6812MINI-E_3.2x2.8mm_P1.5mm_ReverseMount, F.Cu at (-34.5, 240.7)
- added LED278: SK6812MINI-E, LED_SMD:LED_SK6812MINI-E_3.2x2.8mm_P1.5mm_ReverseMount, F.Cu at (-34.5, 245.5)
- added LED279: SK6812MINI-E, LED_SMD:LED_SK6812MINI-E_3.2x2.8mm_P1.5mm_ReverseMount, B.Cu at (193.3, 174.7)
- added LED280: SK6812MINI-E, LED_SMD:LED_SK6812MINI-E_3.2x2.8mm_P1.5mm_ReverseMount, F.Cu at (-9.51, 199.4)
- added LED281: SK6812MINI-E, LED_SMD:LED_SK6812MINI-E_3.2x2.8mm_P1.5mm_ReverseMount, B.Cu at (231.4, 174.7)
- added LED282: SK6812MINI-E, LED_SMD:LED_SK6812MINI-E_3.2x2.8mm_P1.5mm_ReverseMount, F.Cu at (-26.1, 201.7)
- added LED283: SK6812MINI-E, LED_SMD:LED_SK6812MINI-E_3.2x2.8mm_P1.5mm_ReverseMount, F.Cu at (-26.1, 206.6)
- added LED284: SK6812MINI-E, LED_SMD:LED_SK6812MINI-E_3.2x2.8mm_P1.5mm_ReverseMount, F.Cu at (-26.1, 211.5)
- added LED285: SK6812MINI-E, LED_SMD:LED_SK6812MINI-E_3.2x2.8mm_P1.5mm_ReverseMount, F.Cu at (-26.1, 216.3)
- added LED286: SK6812MINI-E, LED_SMD:LED_SK6812MINI-E_3.2x2.8mm_P1.5mm_ReverseMount, F.Cu at (-26.1, 221.2)
- added LED287: SK6812MINI-E, LED_SMD:LED_SK6812MINI-E_3.2x2.8mm_P1.5mm_ReverseMount, F.Cu at (-26.1, 226.1)
- added LED288: SK6812MINI-E, LED_SMD:LED_SK6812MINI-E_3.2x2.8mm_P1.5mm_ReverseMount, F.Cu at (-26.1, 230.9)
- added LED289: SK6812MINI-E, LED_SMD:LED_SK6812MINI-E_3.2x2.8mm_P1.5mm_ReverseMount, F.Cu at (-26.1, 235.8)
- added LED290: SK6812MINI-E, LED_SMD:LED_SK6812MINI-E_3.2x2.8mm_P1.5mm_ReverseMount, F.Cu at (-26.1, 240.7)
- added R101: 33R, Resistor_SMD:R_0603_1608Metric, F.Cu at (166.0, 218.1)
- added R102: 1k, Resistor_SMD:R_0603_1608Metric, F.Cu at (166.0, 220.7)
- added R103: 27R, Resistor_SMD:R_0603_1608Metric, F.Cu at (166.0, 223.2)
- added R104: 27R, Resistor_SMD:R_0603_1608Metric, F.Cu at (170.1, 208.1)
- added R105: 0R, Resistor_SMD:R_0603_1608Metric, F.Cu at (170.1, 210.6)
- added R106: 1k, Resistor_SMD:R_0603_1608Metric, F.Cu at (170.1, 213.1)
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Routing:
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Other:
- copper layers 2 -> 4

Commit message: A
Parts:
- added J101: USB_C_Receptacle_USB2.0_16P, Connector_USB:USB_C_Receptacle_GCT_USB4105-xx-A_16P_TopMnt_Horizontal, F.Cu at (312.5, 63.4)
- added L101: 3u3, Inductor_SMD:L_0805_2012Metric, F.Cu at (343.8, 67.1)
- C101, C102, C103, C104, C105, C106, C107, C108, C109, C110, C111, C112, C113, C114, C115, C116, R101: moved to B.Cu
- moved C102 249.7 mm to (365.2, 71.1)
- moved C101 249.7 mm to (365.2, 68.6)
- moved C104 247.6 mm to (353.5, 63.6), turned to 90 degrees
- moved C103 247.4 mm to (355.2, 63.6), turned to 90 degrees
- moved C109 243.6 mm to (365.2, 76.2)
- moved C106 243.0 mm to (356.7, 80.7), turned to -90 degrees
- moved C107 242.2 mm to (353.9, 80.7), turned to -90 degrees
- moved C113 241.0 mm to (358.3, 80.7), turned to -90 degrees
- moved C115 240.8 mm to (365.2, 72.6)
- moved C116 240.7 mm to (356.7, 63.6), turned to 90 degrees
- moved C105 239.5 mm to (346.7, 70.6), turned to 180 degrees
- moved C114 238.2 mm to (346.7, 72.6), turned to 180 degrees
- moved C108 227.8 mm to (346.7, 74.6), turned to 180 degrees
- moved C112 226.6 mm to (334.3, 71.0)
- moved R101 225.2 mm to (334.3, 68.5)
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Connections:
- D201 pad 1: /Key Matrix/ROW0 -> /Controller/ROW0
- D202 pad 1: /Key Matrix/ROW0 -> /Controller/ROW0
- D203 pad 1: /Key Matrix/ROW0 -> /Controller/ROW0
- D204 pad 1: /Key Matrix/ROW0 -> /Controller/ROW0
- D205 pad 1: /Key Matrix/ROW0 -> /Controller/ROW0
- D206 pad 1: /Key Matrix/ROW0 -> /Controller/ROW0
- D207 pad 1: /Key Matrix/ROW0 -> /Controller/ROW0
- D208 pad 1: /Key Matrix/ROW0 -> /Controller/ROW0
- D209 pad 1: /Key Matrix/ROW0 -> /Controller/ROW0
- D210 pad 1: /Key Matrix/ROW0 -> /Controller/ROW0
- D211 pad 1: /Key Matrix/ROW0 -> /Controller/ROW0
- D212 pad 1: /Key Matrix/ROW0 -> /Controller/ROW0
- D213 pad 1: /Key Matrix/ROW0 -> /Controller/ROW0
- D214 pad 1: /Key Matrix/ROW0 -> /Controller/ROW0
- D215 pad 1: /Key Matrix/ROW0 -> /Controller/ROW0
- D216 pad 1: /Key Matrix/ROW1 -> /Controller/ROW1
- D217 pad 1: /Key Matrix/ROW1 -> /Controller/ROW1
- D218 pad 1: /Key Matrix/ROW1 -> /Controller/ROW1
- D219 pad 1: /Key Matrix/ROW1 -> /Controller/ROW1
- D220 pad 1: /Key Matrix/ROW1 -> /Controller/ROW1
- D221 pad 1: /Key Matrix/ROW1 -> /Controller/ROW1
- D222 pad 1: /Key Matrix/ROW1 -> /Controller/ROW1
- D223 pad 1: /Key Matrix/ROW1 -> /Controller/ROW1
- D224 pad 1: /Key Matrix/ROW1 -> /Controller/ROW1
- D225 pad 1: /Key Matrix/ROW1 -> /Controller/ROW1
- D226 pad 1: /Key Matrix/ROW1 -> /Controller/ROW1
- D227 pad 1: /Key Matrix/ROW1 -> /Controller/ROW1
- D228 pad 1: /Key Matrix/ROW1 -> /Controller/ROW1
- D229 pad 1: /Key Matrix/ROW1 -> /Controller/ROW1
- D230 pad 1: /Key Matrix/ROW1 -> /Controller/ROW1
- D231 pad 1: /Key Matrix/ROW2 -> /Controller/ROW2
- D232 pad 1: /Key Matrix/ROW2 -> /Controller/ROW2
- D233 pad 1: /Key Matrix/ROW2 -> /Controller/ROW2
- D234 pad 1: /Key Matrix/ROW2 -> /Controller/ROW2
- D235 pad 1: /Key Matrix/ROW2 -> /Controller/ROW2
- D236 pad 1: /Key Matrix/ROW2 -> /Controller/ROW2
- D237 pad 1: /Key Matrix/ROW2 -> /Controller/ROW2
- D238 pad 1: /Key Matrix/ROW2 -> /Controller/ROW2
- D239 pad 1: /Key Matrix/ROW2 -> /Controller/ROW2
- D240 pad 1: /Key Matrix/ROW2 -> /Controller/ROW2
- D241 pad 1: /Key Matrix/ROW2 -> /Controller/ROW2
- D242 pad 1: /Key Matrix/ROW2 -> /Controller/ROW2
- D243 pad 1: /Key Matrix/ROW2 -> /Controller/ROW2
- D244 pad 1: /Key Matrix/ROW2 -> /Controller/ROW2
- D245 pad 1: /Key Matrix/ROW2 -> /Controller/ROW2
- D246 pad 1: /Key Matrix/ROW3 -> /Controller/ROW3
- D247 pad 1: /Key Matrix/ROW3 -> /Controller/ROW3
- D248 pad 1: /Key Matrix/ROW3 -> /Controller/ROW3
- D249 pad 1: /Key Matrix/ROW3 -> /Controller/ROW3
- D250 pad 1: /Key Matrix/ROW3 -> /Controller/ROW3
- D251 pad 1: /Key Matrix/ROW3 -> /Controller/ROW3
- D252 pad 1: /Key Matrix/ROW3 -> /Controller/ROW3
- D253 pad 1: /Key Matrix/ROW3 -> /Controller/ROW3
- D254 pad 1: /Key Matrix/ROW3 -> /Controller/ROW3
- D255 pad 1: /Key Matrix/ROW3 -> /Controller/ROW3
- D256 pad 1: /Key Matrix/ROW3 -> /Controller/ROW3
- D257 pad 1: /Key Matrix/ROW3 -> /Controller/ROW3
- D258 pad 1: /Key Matrix/ROW3 -> /Controller/ROW3
- D259 pad 1: /Key Matrix/ROW3 -> /Controller/ROW3
- D260 pad 1: /Key Matrix/ROW3 -> /Controller/ROW3
- D261 pad 1: /Key Matrix/ROW4 -> /Controller/ROW4
- D262 pad 1: /Key Matrix/ROW4 -> /Controller/ROW4
- D263 pad 1: /Key Matrix/ROW4 -> /Controller/ROW4
- D264 pad 1: /Key Matrix/ROW4 -> /Controller/ROW4
- D265 pad 1: /Key Matrix/ROW4 -> /Controller/ROW4
- D266 pad 1: /Key Matrix/ROW4 -> /Controller/ROW4
- D267 pad 1: /Key Matrix/ROW4 -> /Controller/ROW4
- D268 pad 1: /Key Matrix/ROW4 -> /Controller/ROW4
- D269 pad 1: /Key Matrix/ROW4 -> /Controller/ROW4
- D270 pad 1: /Key Matrix/ROW4 -> /Controller/ROW4
- D271 pad 1: /Key Matrix/ROW4 -> /Controller/ROW4
- D272 pad 1: /Key Matrix/ROW4 -> /Controller/ROW4
- D273 pad 1: /Key Matrix/ROW4 -> /Controller/ROW4
- D274 pad 1: /Key Matrix/ROW4 -> /Controller/ROW4
- D275 pad 1: /Key Matrix/ROW4 -> /Controller/ROW4
- SW201 pad 1: /Key Matrix/COL0 -> /Controller/COL0
- SW202 pad 1: /Key Matrix/COL1 -> /Controller/COL1
- SW203 pad 1: /Key Matrix/COL2 -> /Controller/COL2
- SW204 pad 1: /Key Matrix/COL3 -> /Controller/COL3
- SW205 pad 1: /Key Matrix/COL4 -> /Controller/COL4
- SW206 pad 1: /Key Matrix/COL5 -> /Controller/COL5
- SW207 pad 1: /Key Matrix/COL6 -> /Controller/COL6
- SW208 pad 1: /Key Matrix/COL7 -> /Controller/COL7
- SW209 pad 1: /Key Matrix/COL8 -> /Controller/COL8
- SW210 pad 1: /Key Matrix/COL9 -> /Controller/COL9
- SW211 pad 1: /Key Matrix/COL10 -> /Controller/COL10
- SW212 pad 1: /Key Matrix/COL11 -> /Controller/COL11
- SW213 pad 1: /Key Matrix/COL12 -> /Controller/COL12
- SW214 pad 1: /Key Matrix/COL13 -> /Controller/COL13
- SW215 pad 1: /Key Matrix/COL14 -> /Controller/COL14
- SW216 pad 1: /Key Matrix/COL0 -> /Controller/COL0
- SW217 pad 1: /Key Matrix/COL1 -> /Controller/COL1
- SW218 pad 1: /Key Matrix/COL2 -> /Controller/COL2
- SW219 pad 1: /Key Matrix/COL3 -> /Controller/COL3
- SW220 pad 1: /Key Matrix/COL4 -> /Controller/COL4
- SW221 pad 1: /Key Matrix/COL5 -> /Controller/COL5
- SW222 pad 1: /Key Matrix/COL6 -> /Controller/COL6
- SW223 pad 1: /Key Matrix/COL7 -> /Controller/COL7
- SW224 pad 1: /Key Matrix/COL8 -> /Controller/COL8
- SW225 pad 1: /Key Matrix/COL9 -> /Controller/COL9
- SW226 pad 1: /Key Matrix/COL10 -> /Controller/COL10
- SW227 pad 1: /Key Matrix/COL11 -> /Controller/COL11
- SW228 pad 1: /Key Matrix/COL12 -> /Controller/COL12
- SW229 pad 1: /Key Matrix/COL13 -> /Controller/COL13
- SW230 pad 1: /Key Matrix/COL14 -> /Controller/COL14
- SW231 pad 1: /Key Matrix/COL0 -> /Controller/COL0
- SW232 pad 1: /Key Matrix/COL1 -> /Controller/COL1
- SW233 pad 1: /Key Matrix/COL2 -> /Controller/COL2
- SW234 pad 1: /Key Matrix/COL3 -> /Controller/COL3
- SW235 pad 1: /Key Matrix/COL4 -> /Controller/COL4
- SW236 pad 1: /Key Matrix/COL5 -> /Controller/COL5
- SW237 pad 1: /Key Matrix/COL6 -> /Controller/COL6
- SW238 pad 1: /Key Matrix/COL7 -> /Controller/COL7
- SW239 pad 1: /Key Matrix/COL8 -> /Controller/COL8
- SW240 pad 1: /Key Matrix/COL9 -> /Controller/COL9
- SW241 pad 1: /Key Matrix/COL10 -> /Controller/COL10
- SW242 pad 1: /Key Matrix/COL11 -> /Controller/COL11
- SW243 pad 1: /Key Matrix/COL12 -> /Controller/COL12
- SW244 pad 1: /Key Matrix/COL13 -> /Controller/COL13
- SW245 pad 1: /Key Matrix/COL14 -> /Controller/COL14
- SW246 pad 1: /Key Matrix/COL0 -> /Controller/COL0
- SW247 pad 1: /Key Matrix/COL1 -> /Controller/COL1
- SW248 pad 1: /Key Matrix/COL2 -> /Controller/COL2
- SW249 pad 1: /Key Matrix/COL3 -> /Controller/COL3
- SW250 pad 1: /Key Matrix/COL4 -> /Controller/COL4
- SW251 pad 1: /Key Matrix/COL5 -> /Controller/COL5
- SW252 pad 1: /Key Matrix/COL6 -> /Controller/COL6
- SW253 pad 1: /Key Matrix/COL7 -> /Controller/COL7
- SW254 pad 1: /Key Matrix/COL8 -> /Controller/COL8
- SW255 pad 1: /Key Matrix/COL9 -> /Controller/COL9
- SW256 pad 1: /Key Matrix/COL10 -> /Controller/COL10
- SW257 pad 1: /Key Matrix/COL11 -> /Controller/COL11
- SW258 pad 1: /Key Matrix/COL12 -> /Controller/COL12
- SW259 pad 1: /Key Matrix/COL13 -> /Controller/COL13
- SW260 pad 1: /Key Matrix/COL14 -> /Controller/COL14
- SW261 pad 1: /Key Matrix/COL0 -> /Controller/COL0
- SW262 pad 1: /Key Matrix/COL1 -> /Controller/COL1
- SW263 pad 1: /Key Matrix/COL2 -> /Controller/COL2
- SW264 pad 1: /Key Matrix/COL3 -> /Controller/COL3
- SW265 pad 1: /Key Matrix/COL4 -> /Controller/COL4
- SW266 pad 1: /Key Matrix/COL5 -> /Controller/COL5
- SW267 pad 1: /Key Matrix/COL6 -> /Controller/COL6
- SW268 pad 1: /Key Matrix/COL7 -> /Controller/COL7
- SW269 pad 1: /Key Matrix/COL8 -> /Controller/COL8
- SW270 pad 1: /Key Matrix/COL9 -> /Controller/COL9
- SW271 pad 1: /Key Matrix/COL10 -> /Controller/COL10
- SW272 pad 1: /Key Matrix/COL11 -> /Controller/COL11
- SW273 pad 1: /Key Matrix/COL12 -> /Controller/COL12
- SW274 pad 1: /Key Matrix/COL13 -> /Controller/COL13
- SW275 pad 1: /Key Matrix/COL14 -> /Controller/COL14
- U102 pad 20: /Controller/GPIO20 -> /Controller/COL0
- U102 pad 21: /Controller/GPIO21 -> /Controller/COL1
- U102 pad 22: /Controller/GPIO22 -> /Controller/COL2
- U102 pad 23: /Controller/GPIO23 -> /Controller/COL3
- U102 pad 25: /Controller/GPIO24 -> /Controller/COL4
- U102 pad 26: /Controller/GPIO25 -> /Controller/COL5
- U102 pad 27: /Controller/GPIO26 -> /Controller/COL6
- U102 pad 28: /Controller/GPIO27 -> /Controller/COL7
- U102 pad 3: /Controller/GPIO6 -> /Controller/ROW0
- U102 pad 30: unconnected-(U102-XIN-Pad30) -> /Controller/XIN
- U102 pad 31: unconnected-(U102-XOUT-Pad31) -> /Controller/XOUT
- U102 pad 33: unconnected-(U102-SWCLK-Pad33) -> /Controller/SWCLK
- U102 pad 34: unconnected-(U102-SWDIO-Pad34) -> /Controller/SWDIO
- U102 pad 36: /Controller/GPIO28 -> /Controller/COL8
- U102 pad 37: /Controller/GPIO29 -> /Controller/COL9
- U102 pad 38: /Controller/GPIO30 -> /Controller/COL10
- U102 pad 39: /Controller/GPIO31 -> /Controller/COL11
- U102 pad 4: /Controller/GPIO7 -> /Controller/ROW1
- U102 pad 40: /Controller/GPIO32 -> /Controller/COL12
- U102 pad 42: /Controller/GPIO33 -> /Controller/COL13
- U102 pad 43: /Controller/GPIO34 -> /Controller/COL14
- U102 pad 49: unconnected-(U102-GPIO40/ADC0-Pad49) -> /Controller/GPIO40/ADC0
- U102 pad 52: unconnected-(U102-GPIO41/ADC1-Pad52) -> /Controller/GPIO41/ADC1
- U102 pad 53: unconnected-(U102-GPIO42/ADC2-Pad53) -> /Controller/GPIO42/ADC2
- U102 pad 54: unconnected-(U102-GPIO43/ADC3-Pad54) -> /Controller/GPIO43/ADC3
- U102 pad 55: unconnected-(U102-GPIO44/ADC4-Pad55) -> /Controller/GPIO44/ADC4
- U102 pad 56: unconnected-(U102-GPIO45/ADC5-Pad56) -> /Controller/GPIO45/ADC5
- U102 pad 57: unconnected-(U102-GPIO46/ADC6-Pad57) -> /Controller/GPIO46/ADC6
- U102 pad 58: unconnected-(U102-GPIO47/ADC7-Pad58) -> /Controller/GPIO47/ADC7
- U102 pad 6: /Controller/GPIO8 -> /Controller/ROW2
- U102 pad 7: /Controller/GPIO9 -> /Controller/ROW3
- U102 pad 8: /Controller/GPIO10 -> /Controller/ROW4

Commit message: A
Parts:
- removed C101, C110, C111, C112, C113: 4u7, Capacitor_SMD:C_0603_1608Metric
- removed C102, C103, C104, C105, C106, C107, C108, C109, C114, C115, C116, C117, C118: 100n, Capacitor_SMD:C_0603_1608Metric
- removed L101: 3u3, Inductor_SMD:L_0805_2012Metric
- removed R101: 33R, Resistor_SMD:R_0603_1608Metric
- removed R102, R106, R107: 1k, Resistor_SMD:R_0603_1608Metric
- removed R103, R104: 27R, Resistor_SMD:R_0603_1608Metric
- removed R105: 0R, Resistor_SMD:R_0603_1608Metric
- removed SW101: SW_Push, Button_Switch_THT:SW_PUSH_6mm
- removed U101, U103: W25Q128JVS, Package_SO:SOIC-8_5.3x5.3mm_P1.27mm
- removed U102: RP2354B, Package_DFN_QFN:QFN-80-1EP_10x10mm_P0.4mm_EP3.4x3.4mm_ThermalVias
- J101: value USB_C_Receptacle_USB2.0_16P -> Conn_02x20_Top_Bottom; footprint Connector_USB:USB_C_Receptacle_GCT_USB4105-xx-A_16P_TopMnt_Horizontal -> Connector_PinHeader_2.54mm:PinHeader_2x20_P2.54mm_Vertical
- LED283, LED284, LED285, LED286, LED287, LED288: moved to B.Cu
- moved LED288 388.1 mm to (329.1, 74.7), turned to -90 degrees
- moved LED287 381.7 mm to (324.2, 74.7), turned to -90 degrees
- moved LED286 375.3 mm to (319.4, 74.7), turned to -90 degrees
- moved LED285 368.9 mm to (314.5, 74.7), turned to -90 degrees
- moved LED284 362.5 mm to (309.6, 74.7), turned to -90 degrees
- moved LED283 356.2 mm to (304.8, 74.7), turned to -90 degrees
- moved R202 176.3 mm to (-17.9, 246.9)
- moved LED282 19.3 mm to (-9.01, 192.7)
- moved J101 10.9 mm to (307.3, 72.9), turned to 90 degrees
