File: Hardware/PCB/Mk1/Rev1/KBUltraMk1/KBUltraMk1.kicad_pcb (KiCad board)
At the start: 4 copper layers, 310 x 125 mm, 332 parts, among them J101 Conn_02x20_Top_Bottom, SW201 SW_SPST, SW202 SW_SPST, SW203 SW_SPST, SW204 SW_SPST, SW205 SW_SPST, SW206 SW_SPST, SW207 SW_SPST, SW208 SW_SPST, SW209 SW_SPST, SW210 SW_SPST, SW211 SW_SPST, SW212 SW_SPST, SW213 SW_SPST, SW214 SW_SPST, SW215 SW_SPST, SW216 SW_SPST, SW217 SW_SPST, SW218 SW_SPST, SW219 SW_SPST, SW220 SW_SPST, SW221 SW_SPST, SW222 SW_SPST, SW223 SW_SPST, SW224 SW_SPST, SW225 SW_SPST, SW226 SW_SPST, SW227 SW_SPST, SW228 SW_SPST, SW229 SW_SPST, SW230 SW_SPST, SW231 SW_SPST, SW232 SW_SPST, SW233 SW_SPST, SW234 SW_SPST, SW235 SW_SPST, SW236 SW_SPST, SW237 SW_SPST, SW238 SW_SPST, SW239 SW_SPST, SW240 SW_SPST, SW241 SW_SPST, SW242 SW_SPST, SW243 SW_SPST, SW244 SW_SPST, SW245 SW_SPST, SW246 SW_SPST, SW247 SW_SPST, SW248 SW_SPST, SW249 SW_SPST, SW250 SW_SPST, SW251 SW_SPST, SW252 SW_SPST, SW253 SW_SPST, SW254 SW_SPST, SW255 SW_SPST, SW256 SW_SPST, SW257 SW_SPST, SW258 SW_SPST, SW259 SW_SPST, SW260 SW_SPST, SW261 SW_SPST, SW262 SW_SPST, SW263 SW_SPST, SW264 SW_SPST, SW265 SW_SPST, SW266 SW_SPST, SW267 SW_SPST, SW268 SW_SPST, SW269 SW_SPST, SW270 SW_SPST, SW271 SW_SPST, SW272 SW_SPST, SW273 SW_SPST, SW274 SW_SPST, SW275 SW_SPST

Commit message: A
Parts:
- moved C284 67.7 mm to (365.0, 80.9), turned to -90 degrees
- moved C283 66.6 mm to (362.5, 80.9), turned to -90 degrees
- moved C287 60.5 mm to (337.4, 76.9), turned to -90 degrees
- moved C288 59.6 mm to (339.9, 76.9), turned to -90 degrees
- moved C285 57.6 mm to (356.0, 75.9), turned to -90 degrees
- moved C286 48.1 mm to (360.8, 67.7), turned to -90 degrees
Routing:
- net +5V: track 57.9 -> 1618.0 mm, vias 15 -> 20
- net /Controller/ROW3: track 352.3 -> 341.0 mm
- net /Controller/COL10: track 206.4 -> 214.5 mm
- net /Controller/COL3: track 163.1 -> 170.5 mm
- net /Controller/COL9: track 188.4 -> 195.2 mm
- net /Controller/ROW2: track 363.9 -> 357.4 mm
- net /Controller/COL4: track 158.8 -> 163.9 mm
- net /Controller/ROW4: track 426.2 -> 421.4 mm
- net /Controller/COL5: track 164.1 -> 168.2 mm
- net /Controller/COL1: track 159.8 -> 163.5 mm
- net /Controller/COL7: track 394.2 -> 397.3 mm
- net /Controller/COL2: track 159.7 -> 162.2 mm
- net /Controller/COL13: track 87.7 -> 89.5 mm
- net /Controller/COL8: track 402.7 -> 404.4 mm
- net /Controller/COL11: track 260.6 -> 262.1 mm
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- removed copper zone on In1.Cu, net +5V
- removed copper zone on In2.Cu, net +5V
Other:
- copper layers 4 -> 2
