File: Hardware/PCB/Mk1/Rev1/KBUltraMk1/KBUltraMk1.kicad_pcb (KiCad board)
At the start: 2 copper layers, 310 x 125 mm, 324 parts, among them J101 Conn_02x20_Top_Bottom, SW101 RotaryEncoder_Switch, SW201 SW_SPST, SW202 SW_SPST, SW203 SW_SPST, SW204 SW_SPST, SW205 SW_SPST, SW206 SW_SPST, SW207 SW_SPST, SW208 SW_SPST, SW209 SW_SPST, SW210 SW_SPST, SW211 SW_SPST, SW212 SW_SPST, SW213 SW_SPST, SW214 SW_SPST, SW215 SW_SPST, SW216 SW_SPST, SW217 SW_SPST, SW218 SW_SPST, SW219 SW_SPST, SW220 SW_SPST, SW221 SW_SPST, SW222 SW_SPST, SW223 SW_SPST, SW224 SW_SPST, SW225 SW_SPST, SW226 SW_SPST, SW227 SW_SPST, SW228 SW_SPST, SW229 SW_SPST, SW230 SW_SPST, SW231 SW_SPST, SW232 SW_SPST, SW233 SW_SPST, SW234 SW_SPST, SW235 SW_SPST, SW236 SW_SPST, SW237 SW_SPST, SW238 SW_SPST, SW239 SW_SPST, SW240 SW_SPST, SW241 SW_SPST, SW242 SW_SPST, SW243 SW_SPST, SW244 SW_SPST, SW245 SW_SPST, SW246 SW_SPST, SW247 SW_SPST, SW248 SW_SPST, SW249 SW_SPST, SW250 SW_SPST, SW251 SW_SPST, SW252 SW_SPST, SW253 SW_SPST, SW254 SW_SPST, SW255 SW_SPST, SW256 SW_SPST, SW257 SW_SPST, SW258 SW_SPST, SW259 SW_SPST, SW260 SW_SPST, SW261 SW_SPST, SW262 SW_SPST, SW263 SW_SPST, SW264 SW_SPST, SW265 SW_SPST, SW266 SW_SPST, SW267 SW_SPST, SW268 SW_SPST, SW269 SW_SPST, SW270 SW_SPST, SW271 SW_SPST, SW272 SW_SPST, SW273 SW_SPST, SW274 SW_SPST, SW275 SW_SPST, U101 DRV2605LDGS, U102 BMI160, U103 CR2013-MI2120

Commit message: A
Parts:
- added U104: DRV2605LDGS, Package_SO:TSSOP-10_3x3mm_P0.5mm, B.Cu at (88.4, 65.5)
- added U105: DRV2605LDGS, Package_SO:TSSOP-10_3x3mm_P0.5mm, B.Cu at (364.1, 151.2)
- added U106: DRV2605LDGS, Package_SO:TSSOP-10_3x3mm_P0.5mm, B.Cu at (70.9, 168.9)
- U101, U102: moved to B.Cu
- moved U102 113.3 mm to (304.5, 80.9), turned to 180 degrees
- moved U103 82.0 mm to (322.2, 77.4), turned to 90 degrees
- moved U101 58.8 mm to (360.1, 80.5), turned to 180 degrees
Routing:
- net +5V: track 2373.2 -> 2389.5 mm
- net /Controller/POWER_AUX: track 0.00 -> 2.54 mm
- net /Controller/BATT_OUT: track 0.00 -> 2.54 mm
- net Net-(LED201-DOUT): track 53.2 -> 54.7 mm
- net /Controller/COL7: track 401.9 -> 401.2 mm
- net /Controller/COL13: track 280.1 -> 279.5 mm
