File: Hardware/PCB/Mk1/Rev1/KBUltraMk1/controller.kicad_sch (KiCad schematic)
At the start: 31 parts, among them SW101 SW_Push, U101 W25Q128JVS, U102 RP2354B, U103 W25Q128JVS

Commit message: A
Parts:
- L101: footprint (none) -> Inductor_SMD:L_0805_2012Metric
- gave numbers to parts that had none: 1
Changed lines of the file:
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@@
 		(in_pos_files yes)
 		(dnp no)
-		(property "Reference" "J?"
+		(property "Reference" "J101"
 			(at 264.16 20.32 0)
 			(show_name no)
@@
 			(project "KBUltraMk1"
 				(path "/b5c66110-c4bc-44b7-b74f-0bc521af7455/aecb405b-8b8b-4d2e-ac62-4bd044d58a6c"
-					(reference "J?")
+					(reference "J101")
 					(unit 1)
 				)
@@
 			)
 		)
-		(property "Footprint" ""
+		(property "Footprint" "Inductor_SMD:L_0805_2012Metric"
 			(at 43.18 41.91 0)
 			(hide yes)

Commit message: A
Parts:
- removed C101, C110, C111, C112, C113: 4u7, Capacitor_SMD:C_0603_1608Metric, symbol Device:C
- removed C102, C103, C104, C105, C106, C107, C108, C109, C114, C115, C116, C117, C118: 100n, Capacitor_SMD:C_0603_1608Metric, symbol Device:C
- removed J101: USB_C_Receptacle_USB2.0_16P, Connector_USB:USB_C_Receptacle_GCT_USB4105-xx-A_16P_TopMnt_Horizontal, symbol Connector:USB_C_Receptacle_USB2.0_16P
- removed L101: 3u3, Inductor_SMD:L_0805_2012Metric, symbol Device:L
- removed R101: 33R, Resistor_SMD:R_0603_1608Metric, symbol Device:R
- removed R102, R106, R107: 1k, Resistor_SMD:R_0603_1608Metric, symbol Device:R
- removed R103, R104: 27R, Resistor_SMD:R_0603_1608Metric, symbol Device:R
- removed R105: 0R, Resistor_SMD:R_0603_1608Metric, symbol Device:R
- removed SW101: SW_Push, Button_Switch_THT:SW_PUSH_6mm, symbol Switch:SW_Push
- removed U101, U103: W25Q128JVS, Package_SO:SOIC-8_5.3x5.3mm_P1.27mm, symbol Memory_Flash:W25Q128JVS
- removed U102: RP2354B, Package_DFN_QFN:QFN-80-1EP_10x10mm_P0.4mm_EP3.4x3.4mm_ThermalVias, symbol MCU_RaspberryPi:RP2354B
- added J101: Conn_02x20_Top_Bottom, Connector_PinHeader_2.54mm:PinHeader_2x20_P2.54mm_Vertical, symbol Connector_Generic:Conn_02x20_Top_Bottom
