File: Hardware/PCB/Mk1/Rev1/KBUltraMk1/controller.kicad_sch (KiCad schematic)
At the start: 1 part, among them J101 Conn_02x20_Top_Bottom

Commit message: A
Connections:
- net GND: now reaches J101.1 (Pin_1)
- net GND: now also J101.2 (Pin_2)
- net GPIO30: now reaches J101.10 (Pin_10)
- net GPIO29: now reaches J101.11 (Pin_11)
- net GPIO28: now reaches J101.12 (Pin_12)
- net GPIO27: now reaches J101.13 (Pin_13)
- net GPIO26: now reaches J101.14 (Pin_14)
- net GPIO25: now reaches J101.15 (Pin_15)
- net GPIO24: now reaches J101.16 (Pin_16)
- net GPIO23: now reaches J101.17 (Pin_17)
- net GPIO22: now reaches J101.18 (Pin_18)
- net GPIO21: now reaches J101.19 (Pin_19)
- net GPIO20: now reaches J101.20 (Pin_20)
- net BATT_OUT: now reaches J101.21 (Pin_21)
- net BATT_OUT: now also J101.22 (Pin_22)
- net GPIO35: now reaches J101.23 (Pin_23)
- net GPIO34: now reaches J101.24 (Pin_24)
- net GPIO17: now reaches J101.25 (Pin_25)
- net GPIO16: now reaches J101.26 (Pin_26)
- net GPIO15: now reaches J101.27 (Pin_27)
- net GPIO14: now reaches J101.28 (Pin_28)
- net GPIO13: now reaches J101.29 (Pin_29)
- net +5V: now reaches J101.3 (Pin_3)
- net +5V: now also J101.4 (Pin_4)
- net GPIO12: now reaches J101.30 (Pin_30)
- net GPIO11: now reaches J101.31 (Pin_31)
- net GPIO10: now reaches J101.32 (Pin_32)
- net GPIO44: now reaches J101.33 (Pin_33)
- net GPIO43: now reaches J101.34 (Pin_34)
- net GPIO42: now reaches J101.35 (Pin_35)
- net GPIO4: now reaches J101.36 (Pin_36)
- net GPIO3: now reaches J101.37 (Pin_37)
- net GPIO41: now reaches J101.38 (Pin_38)
- net GPIO1: now reaches J101.39 (Pin_39)
- net GPIO40: now reaches J101.40 (Pin_40)
- net POWER_AUX: now reaches J101.5 (Pin_5)
- net POWER_AUX: now also J101.6 (Pin_6)
- net GPIO33: now reaches J101.7 (Pin_7)
- net GPIO32: now reaches J101.8 (Pin_8)
- net GPIO31: now reaches J101.9 (Pin_9)
Other:
- moved on the sheet: J101

Commit message: A
Changed lines of the file:
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@@
-		)
-	)
-	(label "GPIO[0..47]"
-		(at 176.53 44.45 0)
-		(effects
-			(font
-				(size 1.27 1.27)
-			)
-			(justify left bottom)
 		)
 	)
@@
 		)
 	)
-	(label "GPIO[0..47]"
-		(at 127 44.45 180)
-		(effects
-			(font
-				(size 1.27 1.27)
-			)
-			(justify right bottom)
-		)
-	)
 	(label "GPIO31"
 		(at 158.75 76.2 0)
@@
 		(effects
 			(font
+				(size 1.27 1.27)
+			)
+			(justify left)
+		)
+	)
+	(hierarchical_label "GPIO[0..47]"
+		(shape input)
+		(at 127 44.45 180)
+		(effects
+			(font
+				(size 1.27 1.27)
+			)
+			(justify right)
+		)
+	)
+	(hierarchical_label "GPIO[0..47]"
+		(shape input)
+		(at 176.53 44.45 0)
+		(effects
+			(font
