File: Hardware/PCB/Mk1/Rev1/KBUltraMk1/KBUltraMk1.kicad_sch (KiCad schematic)
At the start: 0 parts

Commit message: A
Connections:
- no-connect marks 0 -> 1
Changed lines of the file:
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@@
 	(generator_version "10.0")
 	(paper "A4")
+	(no_connect
+		(at 226.06 88.9)
+	)
 	(wire
 		(pts
@@
 		)
 		(stroke
+			(width 0)
+			(type default)
+		)
+	)
+	(wire
+		(pts
+			(xy 226.06 88.9) (xy 228.6 88.9)
+		)
+		(stroke

Commit message: A
Other:
- removed sheet Extras
- added sheet Accelerometer (accelerometer.kicad_sch)
- added sheet Encoder (encoder.kicad_sch)
- added sheet Haptic (haptic.kicad_sch)
- added sheet Screen (screen.kicad_sch)
- sheet Controller ports: added GPIO[0..47]; removed none

Commit message: A
Parts:
- added C106, C107: 10u, Capacitor_SMD:C_0603_1608Metric, symbol Device:C
- added C108: 100u, Capacitor_Tantalum_SMD:CP_EIA-3528-21_Kemet-B_HandSolder, symbol Device:C_Polarized
- added D101, D103: BLUE, LED_SMD:LED_0603_1608Metric, symbol Device:LED
- added R106, R107: 10k, Resistor_SMD:R_0603_1608Metric, symbol Device:R
- added U104: AZ1117-3.3, Package_TO_SOT_SMD:SOT-223-3_TabPin2, symbol Regulator_Linear:AZ1117-3.3
Connections:
- new net: D101.2 (A), R106.2
- new net: D103.2 (A), R107.2
- new net +3V3: C107.2, C108.1, R107.1, U104.2 (VO)
- new net +5V: C106.2, R106.1, U104.3 (VI)
- new net GND: C106.1, C107.1, C108.2, D101.1 (K), D103.1 (K), U104.1 (GND)
Other:
- sheet Accelerometer ports: added none; removed INT1, INT2
- sheet Controller ports: added none; removed COL[0..14], ROW[0..4]
- sheet Encoder ports: added ENC_A, ENC_BTN, ENC_C; removed none
- sheet Haptic ports: added IN/TRIG, SCL, SDA; removed none
- sheet Key Matrix ports: added GPIO[0..47]; removed COL[0..14], ROW[0..4]
- sheet Screen ports: added none; removed LED
