File: Hardware/PCB/Mk1/Rev1/KBUltraMk1/accelerometer.kicad_sch (KiCad schematic)
At the start: 0 parts

Commit message: A
Parts:
- added U102: BMI160, Package_LGA:Bosch_LGA-14_3x2.5mm_P0.5mm, symbol Sensor_Motion:BMI160
Other:
- note added: "https://www.digikey.ca/en/products/detail/bosch-sensortec/BMI270/9974486"
Changed lines of the file:
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@@
 	(generator_version "10.0")
 	(paper "A4")
+	(text "https://www.digikey.ca/en/products/detail/bosch-sensortec/BMI270/9974486"
+		(exclude_from_sim no)
+		(at 112.014 55.88 0)
+		(effects
+			(font
+				(size 1.27 1.27)
+			)
+		)
+	)
+	(symbol
+		(lib_id "Sensor_Motion:BMI160")
+		(at 104.14 77.47 0)
+		(unit 1)
+		(body_style 1)
+		(exclude_from_sim no)
+		(in_bom yes)
+		(on_board yes)
+		(in_pos_files yes)
+		(dnp no)
+		(fields_autoplaced yes)
+		(property "Reference" "U102"
+			(at 106.2833 64.77 0)
+			(show_name no)
+			(do_not_autoplace no)
+			(effects
+				(font
+					(size 1.27 1.27)
+				)
+				(justify left)
+			)
+		)
+		(property "Value" "BMI160"
+			(at 106.2833 67.31 0)
+			(show_name no)
+			(do_not_autoplace no)
+			(effects
+				(font
+					(size 1.27 1.27)
+				)
+				(justify left)
+			)
+		)
+		(property "Footprint" "Package_LGA:Bosch_LGA-14_3x2.5mm_P0.5mm"
+			(at 104.14 77.47 0)
+			(hide yes)
+			(show_name no)
+			(do_not_autoplace no)
+			(effects
+				(font
+					(size 1.27 1.27)
+				)
+			)
+		)
+		(property "Datasheet" "https://www.bosch-sensortec.com/media/boschsensortec/downloads/datasheets/bst-bmi160-ds000.pdf"
+			(at 86.36 55.88 0)
+			(hide yes)
+			(show_name no)
+			(do_not_autoplace no)
+			(effects
+				(font
+					(size 1.27 1.27)
+				)
+			)
+		)
+		(property "Description" "Small, low power inertial measurement unit, LGA-14"
+			(at 104.14 77.47 0)
+			(hide yes)
+			(show_name no)
+			(do_not_autoplace no)
+			(effects
+				(font
+					(size 1.27 1.27)
+				)
+			)
+		)
+		(pin "10"
+		)
+		(pin "2"
+		)
+		(pin "14"
+		)
+		(pin "7"
+		)
+		(pin "4"
+		)
+		(pin "3"
+		)
+		(pin "5"
+		)
+		(pin "6"
+		)
+		(pin "8"
+		)
+		(pin "1"
+		)
+		(pin "9"
+		)
+		(pin "11"
+		)
+		(pin "12"
+		)
+		(pin "13"
+		)
+		(instances
+			(project "KBUltraMk1"
+				(path "/b5c66110-c4bc-44b7-b74f-0bc521af7455/37a2e385-e742-4cdf-beae-5de0108665d5/4088ed00-9493-4f4c-90bf-8af09cea9729"
+					(reference "U102")
+					(unit 1)
+				)
+			)
+		)
+	)
 )

Commit message: A
Connections:
- net SDO: now reaches U102.1 (SDO)
- net OCSB: now reaches U102.10 (OCSB)
- net OSDO: now reaches U102.11 (OSDO)
- net CSB: now reaches U102.12 (CSB)
- net SCx: now reaches U102.13 (SCx)
- net SDx: now reaches U102.14 (SDx)
- net ASDx: now reaches U102.2 (ASDx)
- net ASCx: now reaches U102.3 (ASCx)
- net INT1: now reaches U102.4 (INT1)
- net VDDIO: now reaches U102.5 (VDDIO)
- net GNDIO: now reaches U102.6 (GNDIO)
- net GND: now reaches U102.7 (GND)
- net VDD: now reaches U102.8 (VDD)
- net INT2: now reaches U102.9 (INT2)

Commit message: A
Parts:
- added C110: 10u, Capacitor_SMD:C_0603_1608Metric, symbol Device:C
- added C111: 100n, Capacitor_SMD:C_0603_1608Metric, symbol Device:C
- added R108: 0R, Resistor_SMD:R_0603_1608Metric, symbol Device:R
- added TP101, TP102, TP103, TP104: TestPoint, TestPoint:TestPoint_Pad_D1.0mm, symbol Connector:TestPoint
Connections:
- net GNDIO is gone; now on net GND: U102.6 (GNDIO)
- net VDD is gone; now on net +3V3: U102.8 (VDD)
- net VDDIO is gone; now on net +3V3: U102.5 (VDDIO)
- net ASCx: now also TP102.1
- net ASDx: now also TP101.1
- net GND: now also C110.2, C111.2
- net OCSB: now also TP103.1
- net OSDO: now also TP104.1
- net SDO: now also R108.2
- net CSB renamed +3V3
- net +3V3: now also C110.1, C111.1, R108.1
- net INT1: no longer names the net of U102.4 (INT1)
- net INT2: no longer names the net of U102.9 (INT2)
- no-connect marks 0 -> 2
Other:
- note added: "The I²C addresses are identical to BMG160. The default I²C address of the device is 0b1101000 (0x68). It is used if the SDO pin is pulled to ´GND´. The alternative address 0b1101001 (0x69) is selected by pulling the SDO pin to ´VDDIO´."
