File: Hardware/PCB/Mk1/Rev1/KBUltraMk1/encoder.kicad_sch (KiCad schematic)
At the start: 0 parts

Commit message: A
Parts:
- added SW101: RotaryEncoder_Switch, Rotary_Encoder:RotaryEncoder_Alps_EC11E-Switch_Vertical_H20mm_MountingHoles, symbol Device:RotaryEncoder_Switch
Other:
- note added: "https://www.digikey.ca/en/products/detail/bourns-inc/PEC12R-4220F-S0024/4499653"
Changed lines of the file:
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@@
 	(generator_version "10.0")
 	(paper "A4")
+	(text "https://www.digikey.ca/en/products/detail/bourns-inc/PEC12R-4220F-S0024/4499653"
+		(exclude_from_sim no)
+		(at 92.71 105.664 0)
+		(effects
+			(font
+				(size 1.27 1.27)
+			)
+		)
+	)
+	(symbol
+		(lib_id "Device:RotaryEncoder_Switch")
+		(at 99.06 78.74 0)
+		(unit 1)
+		(body_style 1)
+		(exclude_from_sim no)
+		(in_bom yes)
+		(on_board yes)
+		(in_pos_files yes)
+		(dnp no)
+		(fields_autoplaced yes)
+		(property "Reference" "SW101"
+			(at 99.06 68.58 0)
+			(show_name no)
+			(do_not_autoplace no)
+			(effects
+				(font
+					(size 1.27 1.27)
+				)
+			)
+		)
+		(property "Value" "RotaryEncoder_Switch"
+			(at 99.06 71.12 0)
+			(show_name no)
+			(do_not_autoplace no)
+			(effects
+				(font
+					(size 1.27 1.27)
+				)
+			)
+		)
+		(property "Footprint" "Rotary_Encoder:RotaryEncoder_Alps_EC11E-Switch_Vertical_H20mm_MountingHoles"
+			(at 95.25 74.676 0)
+			(hide yes)
+			(show_name no)
+			(do_not_autoplace no)
+			(effects
+				(font
+					(size 1.27 1.27)
+				)
+			)
+		)
+		(property "Datasheet" ""
+			(at 99.06 72.136 0)
+			(hide yes)
+			(show_name no)
+			(do_not_autoplace no)
+			(effects
+				(font
+					(size 1.27 1.27)
+				)
+			)
+		)
+		(property "Description" "Rotary encoder, dual channel, incremental quadrate outputs, with switch"
+			(at 99.06 78.74 0)
+			(hide yes)
+			(show_name no)
+			(do_not_autoplace no)
+			(effects
+				(font
+					(size 1.27 1.27)
+				)
+			)
+		)
+		(pin "S2"
+		)
+		(pin "C"
+		)
+		(pin "B"
+		)
+		(pin "A"
+		)
+		(pin "S1"
+		)
+		(instances
+			(project "KBUltraMk1"
+				(path "/b5c66110-c4bc-44b7-b74f-0bc521af7455/37a2e385-e742-4cdf-beae-5de0108665d5/90a1a563-c2d3-4256-984f-1f92d92f3ce2"
+					(reference "SW101")
+					(unit 1)
+				)
+			)
+		)
+	)
 )

Commit message: A
Parts:
- added R104, R105: 10k, Resistor_SMD:R_0603_1608Metric, symbol Device:R
Connections:
- net ENC_A: now reaches SW101.A
- net ENC_C: now reaches SW101.B
- net at SW101.C: now also R105.2
- net at SW101.S1: now also R104.1
- net GND: now reaches SW101.S2
- net GND: now also R105.1
- new net ENC_BTN: R104.2
Other:
- moved on the sheet: SW101
