File: Hardware/PCB/Mk1/Rev1/KBUltraMk1/haptic.kicad_sch (KiCad schematic)
At the start: 0 parts

Commit message: A
Parts:
- added M101, M102, M103, M104: Motor_DC_ALT, symbol Motor:Motor_DC_ALT
- added U101: DRV2605LDGS, Package_SO:TSSOP-10_3x3mm_P0.5mm, symbol Driver:DRV2605LDGS

Commit message: A
Parts:
- added U104, U105, U106: DRV2605LDGS, Package_SO:TSSOP-10_3x3mm_P0.5mm, symbol Driver:DRV2605LDGS
Connections:
- net SCL: now reaches U101.2 (SCL)
- net SCL: now also U104.2 (SCL), U105.2 (SCL), U106.2 (SCL)
- net SDA: now reaches U101.3 (SDA)
- net SDA: now also U104.3 (SDA), U105.3 (SDA), U106.3 (SDA)
- net IN/TRIG: now reaches U101.4 (IN/TRIG)
- net IN/TRIG: now also U104.4 (IN/TRIG), U105.4 (IN/TRIG), U106.4 (IN/TRIG)
- net EN: now reaches U101.5 (EN)
- net EN: now also U104.5 (EN), U105.5 (EN), U106.5 (EN)
- net VDD/NC: now reaches U101.6 (VDD/NC)
- net VDD/NC: now also U104.6 (VDD/NC), U105.6 (VDD/NC), U106.6 (VDD/NC)
Other:
- moved on the sheet: U101

Commit message: A
Parts:
- removed M102, M103, M104: Motor_DC_ALT, symbol Motor:Motor_DC_ALT
- removed U104, U105, U106: DRV2605LDGS, Package_SO:TSSOP-10_3x3mm_P0.5mm, symbol Driver:DRV2605LDGS
- added C101: 1u, Capacitor_SMD:C_0603_1608Metric, symbol Device:C
- added C102: 10u, Capacitor_SMD:C_0805_2012Metric, symbol Device:C
- added C109: 100n, Capacitor_SMD:C_0402_1005Metric, symbol Device:C
- added R101, R102, R103: 10k, Resistor_SMD:R_0603_1608Metric, symbol Device:R
- added R110: 0R, Resistor_SMD:R_0603_1608Metric, symbol Device:R
- M101: footprint (none) -> Connector_PinHeader_2.54mm:PinHeader_1x02_P2.54mm_Vertical
Connections:
- net VDD/NC is gone; now on net +3V3: U101.6 (VDD/NC)
- net EN: now also R110.1
- net SCL: now also R103.2
- net SDA: now also R102.2
- net at U101.1 (REG): now also C101.1
- net +3V3: now reaches U101.10 (VDD)
- net +3V3: now also C102.1, C109.1, R102.1, R103.1, R110.2
- net at U101.7 (OUT+): now also M101.1 (+)
- net GND: now reaches U101.8 (GND)
- net GND: now also C101.2, C102.2, C109.2, R101.2
- net at U101.9 (OUT-): now also M101.2 (-)
- net IN/TRIG renamed IN/TRIG
- net IN/TRIG: now also R101.1
Other:
- moved on the sheet: M101, U101
