File: Hardware/PCB/Mk1/Rev1/KBUltraMk1/key_matrix.kicad_sch (KiCad schematic)
At the start: 163 parts, among them SW201 SW_SPST, SW202 SW_SPST, SW203 SW_SPST, SW204 SW_SPST, SW205 SW_SPST, SW206 SW_SPST, SW207 SW_SPST, SW208 SW_SPST, SW209 SW_SPST, SW210 SW_SPST, SW211 SW_SPST, SW212 SW_SPST, SW213 SW_SPST, SW214 SW_SPST, SW215 SW_SPST, SW216 SW_SPST, SW217 SW_SPST, SW218 SW_SPST, SW219 SW_SPST, SW220 SW_SPST, SW221 SW_SPST, SW222 SW_SPST, SW223 SW_SPST, SW224 SW_SPST, SW225 SW_SPST, SW226 SW_SPST, SW227 SW_SPST, SW228 SW_SPST, SW229 SW_SPST, SW230 SW_SPST, SW231 SW_SPST, SW232 SW_SPST, SW233 SW_SPST, SW234 SW_SPST, SW235 SW_SPST, SW236 SW_SPST, SW237 SW_SPST, SW238 SW_SPST, SW239 SW_SPST, SW240 SW_SPST, SW241 SW_SPST, SW242 SW_SPST, SW243 SW_SPST, SW244 SW_SPST, SW245 SW_SPST, SW246 SW_SPST, SW247 SW_SPST, SW248 SW_SPST, SW249 SW_SPST, SW250 SW_SPST, SW251 SW_SPST, SW252 SW_SPST, SW253 SW_SPST, SW254 SW_SPST, SW255 SW_SPST, SW256 SW_SPST, SW257 SW_SPST, SW258 SW_SPST, SW259 SW_SPST, SW260 SW_SPST, SW261 SW_SPST, SW262 SW_SPST, SW263 SW_SPST, SW264 SW_SPST, SW265 SW_SPST, SW266 SW_SPST, SW267 SW_SPST, SW268 SW_SPST, SW269 SW_SPST, SW270 SW_SPST, SW271 SW_SPST, SW272 SW_SPST, SW273 SW_SPST, SW274 SW_SPST, SW275 SW_SPST

Commit message: A
Parts:
- SW201, SW202, SW203, SW204, SW205, SW206, SW207, SW208, SW209, SW210, SW211, SW212, SW213, SW214, SW215, SW216, SW217, SW218, SW219, SW220, SW221, SW222, SW223, SW224, SW226, SW228, SW229, SW230, SW231, SW232, SW233, SW234, SW235, SW236, SW237, SW238, SW239, SW241, SW243, SW244, SW245, SW246, SW247, SW248, SW249, SW250, SW251, SW252, SW253, SW255, SW257, SW258, SW259, SW260, SW261, SW262, SW263, SW264, SW265, SW266: JLC Part# (none) -> C49352235

Commit message: A
Parts:
- D201, D202, D203, D204, D205, D206, D207, D208, D209, D210, D211, D212, D213, D214, D215, D216, D217, D218, D219, D220, D221, D222, D223, D224, D225, D226, D227, D228, D229, D230, D231, D232, D233, D234, D235, D236, D237, D238, D239, D240, D241, D242, D243, D244, D245, D246, D247, D248, D249, D250, D251, D252, D253, D254, D255, D256, D257, D258, D259, D260, D261, D262, D263, D264, D265, D266, D267, D268, D269, D270, D271, D272, D273, D274, D275: JLC Part# (none) -> C81598
- SW201, SW202, SW203, SW204, SW205, SW206, SW207, SW208, SW209, SW210, SW211, SW212, SW213, SW214, SW215, SW216, SW217, SW218, SW219, SW220, SW221, SW222, SW223, SW224, SW226, SW228, SW229, SW230, SW231, SW232, SW233, SW234, SW235, SW236, SW237, SW238, SW239, SW241, SW243, SW244, SW245, SW246, SW247, SW248, SW249, SW250, SW251, SW252, SW253, SW255, SW257, SW258, SW259, SW260, SW261, SW262, SW263, SW264, SW265, SW266: JLC Part# C49352235 -> C41430893
- SW225, SW227, SW240, SW242, SW254, SW256, SW267, SW268, SW269, SW270, SW271, SW272, SW273, SW274, SW275: JLC Part# (none) -> C41430893
Connections:
- net COL0 renamed GPIO12
- net COL1 renamed GPIO13
- net COL10 renamed GPIO31
- net COL11 renamed GPIO32
- net COL12 renamed GPIO33
- net COL13 renamed GPIO41
- net COL14 renamed GPIO44
- net COL2 renamed GPIO14
- net COL3 renamed GPIO15
- net COL4 renamed GPIO17
- net COL5 renamed GPIO20
- net COL6 renamed GPIO21
- net COL7 renamed GPIO22
- net COL8 renamed GPIO24
- net COL9 renamed GPIO30
- net ROW0 renamed GPIO1
- net ROW1 renamed GPIO3
- net ROW2 renamed GPIO4
- net ROW3 renamed GPIO10
- net ROW4 renamed GPIO11
