File: Hardware/PCB/Mk1/Rev1/KBUltraMk1/lighting.kicad_sch (KiCad schematic)
At the start: 168 parts

Commit message: A
Parts:
- removed C283, C284, C285, C286, C287, C288: 100n, Capacitor_SMD:C_0603_1608Metric, symbol Device:C
- removed LED283, LED284, LED285, LED286, LED287, LED288: SK6812MINI-E, LED_SMD:LED_SK6812MINI-E_3.2x2.8mm_P1.5mm_ReverseMount, symbol LED:SK6812MINI-E
Connections:
- net at R202.2: now also LED275.4 (DOUT)
- net at LED271.2 (DIN): now also LED279.4 (DOUT); no longer LED270.4 (DOUT)
- net at LED271.4 (DOUT): now also LED281.2 (DIN); no longer LED272.2 (DIN)
- net at LED279.2 (DIN): now also LED270.4 (DOUT); no longer LED275.4 (DOUT)
- net at LED281.4 (DOUT): now also LED272.2 (DIN)
Other:
- moved on the sheet: LED271, LED272, LED273, LED274, LED275, LED281, R202

Commit message: A
Parts:
- C201, C202, C203, C204, C205, C206, C207, C208, C209, C210, C211, C212, C213, C214, C215, C216, C217, C218, C219, C220, C221, C222, C223, C224, C225, C226, C227, C228, C229, C230, C231, C232, C233, C234, C235, C236, C237, C238, C239, C240, C241, C242, C243, C244, C245, C246, C247, C248, C249, C250, C251, C252, C253, C254, C255, C256, C257, C258, C259, C260, C261, C262, C263, C264, C265, C266, C267, C268, C269, C270, C271, C272, C273, C274, C275, C279, C281: JLC Part# (none) -> C14663
- R201, R202: JLC Part# (none) -> C23193
