File: Hardware/PCB/Mk1/Rev1/KBUltraMk1/screen.kicad_sch (KiCad schematic)
At the start: 0 parts

Commit message: A
Parts:
- added U103: CR2013-MI2120, Display:CR2013-MI2120, symbol Driver_Display:CR2013-MI2120
Connections:
- no-connect marks 0 -> 1
Changed lines of the file:
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@@
 	(generator_version "10.0")
 	(paper "A4")
+	(no_connect
+		(at 128.27 102.87)
+	)
+	(symbol
+		(lib_id "Driver_Display:CR2013-MI2120")
+		(at 121.92 80.01 0)
+		(unit 1)
+		(body_style 1)
+		(exclude_from_sim no)
+		(in_bom yes)
+		(on_board yes)
+		(in_pos_files yes)
+		(dnp no)
+		(fields_autoplaced yes)
+		(property "Reference" "U103"
+			(at 124.0633 62.23 0)
+			(show_name no)
+			(do_not_autoplace no)
+			(effects
+				(font
+					(size 1.27 1.27)
+				)
+				(justify left)
+			)
+		)
+		(property "Value" "CR2013-MI2120"
+			(at 124.0633 64.77 0)
+			(show_name no)
+			(do_not_autoplace no)
+			(effects
+				(font
+					(size 1.27 1.27)
+				)
+				(justify left)
+			)
+		)
+		(property "Footprint" "Display:CR2013-MI2120"
+			(at 121.92 97.79 0)
+			(hide yes)
+			(show_name no)
+			(do_not_autoplace no)
+			(effects
+				(font
+					(size 1.27 1.27)
+				)
+			)
+		)
+		(property "Datasheet" "http://pan.baidu.com/s/11Y990"
+			(at 105.41 67.31 0)
+			(hide yes)
+			(show_name no)
+			(do_not_autoplace no)
+			(effects
+				(font
+					(size 1.27 1.27)
+				)
+			)
+		)
+		(property "Description" "ILI9341 controller, SPI TFT LCD Display, 9-pin breakout PCB, 4-pin SD card interface, 5V/3.3V"
+			(at 121.92 80.01 0)
+			(hide yes)
+			(show_name no)
+			(do_not_autoplace no)
+			(effects
+				(font
+					(size 1.27 1.27)
+				)
+			)
+		)
+		(pin "9"
+		)
+		(pin "11"
+		)
+		(pin "4"
+		)
+		(pin "12"
+		)
+		(pin "8"
+		)
+		(pin "13"
+		)
+		(pin "5"
+		)
+		(pin "1"
+		)
+		(pin "2"
+		)
+		(pin "3"
+		)
+		(pin "6"
+		)
+		(pin "7"
+		)
+		(pin "14"
+		)
+		(pin "10"
+		)
+		(instances
+			(project "KBUltraMk1"
+				(path "/b5c66110-c4bc-44b7-b74f-0bc521af7455/37a2e385-e742-4cdf-beae-5de0108665d5/fbff92d3-74ba-4fa3-9981-79b8655e9aac"
+					(reference "U103")
+					(unit 1)
+				)
+			)
+		)
+	)
 )

Commit message: A
Connections:
- net VCC: now reaches U103.1 (VCC)
- net SD_CS: now reaches U103.10 (SD_CS)
- net SD_MOSI: now reaches U103.11 (SD_MOSI)
- net SD_MISO: now reaches U103.12 (SD_MISO)
- net SD_SCK: now reaches U103.13 (SD_SCK)
- net FLASH_CD: now reaches U103.14 (FLASH_CD)
- net GND: now reaches U103.2 (GND)
- net ~{CS}: now reaches U103.3 (~{CS})
- net RESET: now reaches U103.4 (RESET)
- net D/~{C}: now reaches U103.5 (D/~{C})
- net MOSI: now reaches U103.6 (MOSI)
- net SCK: now reaches U103.7 (SCK)
- net LED: now reaches U103.8 (LED)
- net MISO: now reaches U103.9 (MISO)
- no-connect marks 1 -> 5

Commit message: A
Parts:
- added C103: 10u, Capacitor_SMD:C_0603_1608Metric, symbol Device:C
- added C104: 100n, Capacitor_SMD:C_0603_1608Metric, symbol Device:C
- added C105: 100u, Capacitor_Tantalum_SMD:CP_EIA-3528-21_Kemet-B_HandSolder, symbol Device:C_Polarized
- added JP101: SolderJumper_3_Open, Jumper:SolderJumper-3_P2.0mm_Open_TrianglePad1.0x1.5mm_NumberLabels, symbol Jumper:SolderJumper_3_Open
- added R109: 0R, Resistor_SMD:R_0603_1608Metric, symbol Device:R
Connections:
- net GND: now also C103.2, C104.2, C105.2
- net LED: now also R109.1
- net VCC: no longer names the net of U103.1 (VCC)
- net VCC: now also C103.1, C104.1, C105.1, JP101.2 (C), R109.2
- new net +3V3: JP101.1 (A)
- new net +5V: JP101.3 (B)
