File: ControlCardRP/Hardware/Rev1/ControlCardRP/battery_management.kicad_sch (KiCad schematic)
At the start: 27 parts, among them J4 JST_PK BATTERY, J5 PIN_HEADER BATTERY, U2 BQ24075RGT, U3 BQ27427YZFR

Commit message: A
Parts:
- removed R14: 200k, symbol Device:R
- removed R17, R18, R22, R23: 0R, symbol Device:R
- added C20: 4u7, Capacitor_SMD:C_0402_1005Metric, symbol Device:C
- added R45, R46, R47: 0R, Resistor_SMD:R_0402_1005Metric, symbol Device:R
- added R48, R49: 10k, Resistor_SMD:R_0402_1005Metric, symbol Device:R
- added SW1: SW_SPST, Button_Switch_SMD:SW_SPDT_PCM12, symbol Switch:SW_SPST
- C6, C8: footprint (none) -> Capacitor_SMD:C_0603_1608Metric; LCSC Part # (none) -> C15849
- C7: footprint (none) -> Capacitor_SMD:C_0603_1608Metric; LCSC Part # (none) -> C12530
- C9: value 4u7 -> 10u; footprint (none) -> Capacitor_SMD:C_0603_1608Metric; LCSC Part # (none) -> C440198
- D3, D4: footprint (none) -> LED_SMD:LED_0603_1608Metric
- JP1: footprint (none) -> Jumper:SolderJumper-2_P1.3mm_Open_TrianglePad1.0x1.5mm
- R10: value R -> 1k13; footprint (none) -> Resistor_SMD:R_0402_1005Metric; LCSC Part # (none) -> C25862
- R11: value R -> 1k18; footprint (none) -> Resistor_SMD:R_0402_1005Metric; LCSC Part # (none) -> C25867
- R12, R13: footprint (none) -> Resistor_SMD:R_0402_1005Metric; LCSC Part # (none) -> C25867
- R15, R16: footprint (none) -> Resistor_SMD:R_0402_1005Metric; LCSC Part # (none) -> C17168
- R19, R20: footprint (none) -> Resistor_SMD:R_0402_1005Metric; LCSC Part # (none) -> C25744
- R21: footprint (none) -> Resistor_SMD:R_0402_1005Metric; LCSC Part # (none) -> C25764
- R8: value 49k9 -> 10k; footprint (none) -> Resistor_SMD:R_0402_1005Metric; LCSC Part # (none) -> C25744
- R9: footprint (none) -> Resistor_SMD:R_0402_1005Metric; now not fitted
- U3: footprint DSBGA9-YZF_TEX -> footprints:DSBGA9-YZF_TEX
Connections:
- net BATT_GPOUT: now also R45.2; no longer U3.A1 (GPOUT)
- net BATT_OUT: now also SW1.2 (B)
- net BATT_SCL: now also R47.2; no longer U3.A3 (SCL)
- net BATT_SDA: now also R46.2; no longer U3.A2 (SDA)
- net GND: now also C20.2, R48.1, R49.1
- net SYSOFF: now also R49.2, SW1.1 (A)
- net ~{CE}: now also R48.2
- net VDD: now reaches C7.1, U3.B3 (VDD)
- net at U2.2 (BAT), U2.3 (BAT), U3.C2 (SRX): now also C20.1
- new net: R45.1, U3.A1 (GPOUT)
- new net: R46.1, U3.A2 (SDA)
- new net: R47.1, U3.A3 (SCL)
Other:
- note added: "TMR Safety Timer will be deafult 5Hrs"
- moved on the sheet: C7, R15, R16, R19, R20, R8
