File: ControlCardRP/Hardware/Rev1/ControlCardRP/battery_management.kicad_sch (KiCad schematic)
At the start: 29 parts, among them J4 JST_PK BATTERY, J5 PIN_HEADER BATTERY, SW1 SW_SPDT, U2 BQ24075RGT, U3 BQ27427YZFR

Commit message: A
Parts:
- C9: LCSC Part # C440198 -> C96446
Changed lines of the file:
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@@
 			)
 		)
-		(property "LCSC Part #" "C440198"
+		(property "LCSC Part #" "C96446"
 			(at 107.95 130.81 0)
 			(hide yes)
