File: ControlCardRP/Hardware/Rev1/ControlCardRP/power.kicad_sch (KiCad schematic)
At the start: 1 part, among them U4 TPS63002

Commit message: A
Parts:
- added C10: C, symbol Device:C
- added L1: 2u2, symbol Device:L
- added R24: R, symbol Device:R
Connections:
- net at U4.1 (VOUT): now also U4.10 (FB)
- net GND: now reaches U4.11 (PGND), U4.3 (PGND)
- net GND: now also U4.9 (GND), C10.1
- net at U4.2 (L2): now also L1.1
- net at U4.4 (L1): now also L1.2
- net BATT_OUT: now reaches U4.5 (VIN)
- net BATT_OUT: now also R24.1
- net at U4.6 (EN): now also U4.7 (PS/SYNC), U4.8 (VINA), C10.2, R24.2
