File: ControlCardRP/Hardware/Rev1/ControlCardRP/power.kicad_sch (KiCad schematic)
At the start: 4 parts, among them U4 TPS63002

Commit message: A
Parts:
- removed U4: TPS63002, Package_SON:Texas_DRC0010J_ThermalVias, symbol Regulator_Switching:TPS63002
- added C11, C12, C15, C16, C17: 100n, symbol Device:C
- added C13: 100u, symbol Device:C_Polarized
- added C14: 22n, symbol Device:C
- added C18: 22u, symbol Device:C
- added R26: 430k, symbol Device:R
- added R27: 107k, symbol Device:R
- added R28, R30: 499k, symbol Device:R
- added R29: 806k, symbol Device:R
- added R31, R32: 10k, symbol Device:R
- added U4: MP28167GQ-A-P, footprints:QFN-16_MP28167_MNP, symbol controlboard:MP28167GQ-A-P
- C10: value C -> 100n
- L1: value 2u2 -> 4u7
- R24: value R -> 499k
Connections:
- net GND: now also C12.2, C13.2, C14.2, C15.2, C16.2, C17.2, C18.2, R27.2, R28.2, U4.10 (AGND), U4.11 (GND), U4.2 (GND); no longer C10.1
- net at C10.2: now also U4.13 (BST2); no longer R24.2
- net at L1.1: now also C11.1, U4.15 (SW1)
- net at L1.2: now also C10.1, U4.14 (SW2)
- net BATT_OUT renamed IN
- net IN: now also C12.1, C13.1, U4.1 (IN)
- new net: R26.2, R27.1, R29.1
- new net: C11.2, U4.16 (BST1)
- new net +5V: R31.1, R32.1
- new net ALT: R30.2, U4.4 (ALT)
- new net EN: C14.1, R24.2, U4.3 (EN)
- new net FB: R29.2, U4.8 (FB)
- new net OC: C15.1, R28.1, U4.7 (OC)
- new net OUT: C16.1, C17.1, C18.1, R26.1, U4.12 (OUT)
- new net SCL: R31.2, U4.5 (SCL)
- new net SDA: R32.2, U4.6 (SDA)
- new net VCC: R30.1, U4.9 (VCC)

Commit message: A
Parts:
- removed R31, R32: 10k, symbol Device:R
- added C28: 10u, Capacitor_SMD:C_0402_1005Metric, symbol Device:C
- added D11, D8: LED, LED_SMD:LED_0603_1608Metric, symbol Device:LED
- added R22, R54: 10k, Resistor_SMD:R_0402_1005Metric, symbol Device:R
- added R23, R50, R51, R55: 0R, Resistor_SMD:R_0402_1005Metric, symbol Device:R
- C10, C11, C12, C16, C17: footprint (none) -> Capacitor_SMD:C_0402_1005Metric; LCSC Part # (none) -> C307331
- C13: footprint (none) -> Capacitor_SMD:CP_Elec_5x5.4; now not fitted
- C14: footprint (none) -> Capacitor_SMD:C_0402_1005Metric; LCSC Part # (none) -> C1532
- C15: footprint (none) -> Capacitor_SMD:C_0402_1005Metric; LCSC Part # (none) -> C1525
- C18: footprint (none) -> Capacitor_SMD:C_1206_3216Metric; LCSC Part # (none) -> C12891
- L1: footprint (none) -> Inductor_SMD:L_Taiyo-Yuden_NR-60xx
- R24, R28, R30: footprint (none) -> Resistor_SMD:R_0402_1005Metric; LCSC Part # (none) -> C25778
- R26, R27, R29: footprint (none) -> Resistor_SMD:R_0402_1005Metric; now not fitted
Connections:
- net ALT: now also R55.1
- net EN: now also R51.1
- net GND: now also C28.2, D11.1 (K), D8.1 (K)
- net SCL: now also R23.1
- net SDA: now also R50.1
- net IN renamed POWER_IN
- net POWER_IN: now also C28.1, R22.1
- net OUT renamed POWER_OUT
- net POWER_OUT: now also R54.1
- new net: D11.2 (A), R54.2
- new net: D8.2 (A), R22.2
- new net POWER_ALT: R55.2
- new net POWER_EN: R51.2
- new net POWER_SCL: R23.2
- new net POWER_SDA: R50.2
Other:
- note added: "Only needed if I2C unused."
- note added: "http://digikey.ca/en/products/detail/taiyo-yuden/NRS6028T4R7MMGKV/4693978"
