File: ControlCardRP/Hardware/Rev1/ControlCardRP/power.kicad_sch (KiCad schematic)
At the start: 26 parts, among them U4 MP28167GQ-A-P

Commit message: A
Parts:
- C28: footprint Capacitor_SMD:C_0402_1005Metric -> Capacitor_SMD:C_0603_1608Metric; LCSC Part # C440198 -> C96446
- R26: footprint Resistor_SMD:R_0402_1005Metric -> Resistor_SMD:R_0603_1608Metric; LCSC Part # (none) -> C25969
- R27: footprint Resistor_SMD:R_0402_1005Metric -> Resistor_SMD:R_0603_1608Metric; LCSC Part # (none) -> C25805
- R29: footprint Resistor_SMD:R_0402_1005Metric -> Resistor_SMD:R_0603_1608Metric; LCSC Part # (none) -> C23240
- R55: LCSC Part # (none) -> C17168
Changed lines of the file:
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@@
 			)
 		)
-		(property "LCSC Part #" ""
+		(property "LCSC Part #" "C17168"
 			(at 76.2 175.26 90)
 			(hide yes)
@@
 			)
 		)
-		(property "Footprint" "Resistor_SMD:R_0402_1005Metric"
+		(property "Footprint" "Resistor_SMD:R_0603_1608Metric"
 			(at 111.252 121.92 90)
 			(hide yes)
@@
 			)
 		)
-		(property "LCSC Part #" ""
+		(property "LCSC Part #" "C25805"
 			(at 113.03 121.92 0)
 			(hide yes)
@@
 			)
 		)
-		(property "Footprint" "Capacitor_SMD:C_0402_1005Metric"
+		(property "Footprint" "Capacitor_SMD:C_0603_1608Metric"
 			(at 45.4152 69.85 0)
 			(hide yes)
@@
 			)
 		)
-		(property "LCSC Part #" "C440198"
+		(property "LCSC Part #" "C96446"
 			(at 44.45 66.04 0)
 			(hide yes)
@@
 			)
 		)
-		(property "Footprint" "Resistor_SMD:R_0402_1005Metric"
+		(property "Footprint" "Resistor_SMD:R_0603_1608Metric"
 			(at 111.252 109.22 90)
 			(hide yes)
@@
 			)
 		)
-		(property "LCSC Part #" ""
+		(property "LCSC Part #" "C25969"
 			(at 113.03 109.22 0)
 			(hide yes)
@@
 			)
 		)
-		(property "Footprint" "Resistor_SMD:R_0402_1005Metric"
+		(property "Footprint" "Resistor_SMD:R_0603_1608Metric"
 			(at 124.46 117.348 90)
 			(hide yes)
@@
 			)
 		)
-		(property "LCSC Part #" ""
+		(property "LCSC Part #" "C23240"
 			(at 124.46 115.57 90)
 			(hide yes)
