File: ControlCardRP/Hardware/Rev1/ControlCardRP/usb_c_pd.kicad_sch (KiCad schematic)
At the start: 19 parts, among them J2 USB_C_Receptacle_USB2.0_16P, Q1 NMOS, Q2 NMOS, U1 AP33772SDKZ-xx-FA02

Commit message: A
Connections:
- net PD_OUT renamed VBUS_UCPD
Changed lines of the file:
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@@
 		)
 	)
-	(global_label "PD_OUT"
+	(global_label "VBUS_UCPD"
 		(shape input)
 		(at 205.74 43.18 0)
@@
 		)
 		(property "Intersheetrefs" "${INTERSHEET_REFS}"
-			(at 215.8614 43.18 0)
+			(at 219.7319 43.18 0)
 			(hide yes)
 			(show_name no)
