File: ControlCardRP/Hardware/Rev1/ControlCardRP/usb_c_pd.kicad_sch (KiCad schematic)
At the start: 19 parts, among them J2 USB_C_Receptacle_USB2.0_16P, Q1 NMOS, Q2 NMOS, U1 AP33772SDKZ-xx-FA02

Commit message: A
Parts:
- added R25: 100k, symbol Device:R
Connections:
- net GND: now also R25.1
- net VSEL: now also R25.2
Other:
- note added: "VSEL: Default 5V."
- moved on the sheet: C3, C4, C5, D1, D2, R6, R7, TH1

Commit message: A
Parts:
- added D5: LED, LED_SMD:LED_0603_1608Metric, symbol Device:LED
- added R39: 1k, Resistor_SMD:R_0402_1005Metric, symbol Device:R
- added R40, R41, R42, R43, R44: 0R, Resistor_SMD:R_0402_1005Metric, symbol Device:R
- C1, C4: footprint (none) -> Capacitor_SMD:C_0603_1608Metric; LCSC Part # (none) -> C15849
- C2: footprint (none) -> Capacitor_SMD:C_0603_1608Metric; LCSC Part # (none) -> C440198
- C3, C5: footprint (none) -> Capacitor_SMD:C_0402_1005Metric; LCSC Part # (none) -> C307331
- D1, D2: footprint (none) -> LED_SMD:LED_0603_1608Metric
- Q1, Q2: footprint (none) -> Package_TO_SOT_SMD:SOT-23-3
- R1: footprint (none) -> Resistor_SMD:R_1206_3216Metric
- R2: footprint (none) -> Resistor_SMD:R_0402_1005Metric
- R25, R7: footprint (none) -> Resistor_SMD:R_0402_1005Metric; LCSC Part # (none) -> C25741
- R3, R4: footprint (none) -> Resistor_SMD:R_0402_1005Metric; LCSC Part # (none) -> C25905
- R5: footprint (none) -> Resistor_SMD:R_0402_1005Metric; LCSC Part # (none) -> C25087
- R6: footprint (none) -> Resistor_SMD:R_0402_1005Metric; LCSC Part # (none) -> C11702
- TH1: footprint (none) -> Resistor_SMD:R_0603_1608Metric
Connections:
- net GND: now also D5.1 (K)
- net UCPD_FLIP: now also R44.1; no longer U1.6 (FLIP)
- net UCPD_GPIO: now also R43.1; no longer U1.7 (GPIO)
- net UCPD_INT: now also R42.1; no longer U1.9 (INT)
- net UCPD_SCL: now also R40.1; no longer U1.5 (SCL)
- net UCPD_SDA: now also R41.1; no longer U1.4 (SDA)
- net UCPD_LED renamed LED
- net LED: now also R39.2
- new net: D5.2 (A), R39.1
- new net: R43.2, U1.7 (GPIO)
- new net: R44.2, U1.6 (FLIP)
- new net: R41.2, U1.4 (SDA)
- new net: R40.2, U1.5 (SCL)
- new net: R42.2, U1.9 (INT)
Other:
- note added: "http://digikey.ca/en/products/detail/diodes-incorporated/DMG3406L-7/5223203"
- note added: "https://www.digikey.ca/en/products/detail/ohmite/LVT12R0050FER/9556157"
