File: ControlCardRP/Hardware/Rev1/ControlCardRP/usb_c_pd.kicad_sch (KiCad schematic)
At the start: 27 parts, among them J2 USB_C_Receptacle_USB2.0_16P, Q1 NMOS, Q2 NMOS, U1 AP33772SDKZ-xx-FA02

Commit message: A
Parts:
- C2: LCSC Part # C440198 -> C96446
Changed lines of the file:
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@@
 			)
 		)
-		(property "LCSC Part #" "C440198"
+		(property "LCSC Part #" "C96446"
 			(at 198.12 49.53 0)
 			(hide yes)

Commit message: A
Parts:
- R2: LCSC Part # (none) -> C25905
Changed lines of the file:
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@@
 			)
 		)
-		(property "LCSC Part #" ""
+		(property "LCSC Part #" "C25905"
 			(at 147.32 59.69 0)
 			(hide yes)
