File: ControlCardRP/Hardware/Rev1/ControlCardRP/ControlCardRP.kicad_sch (KiCad schematic)
At the start: 3 parts, among them J1 Conn_02x20_Top_Bottom

Commit message: A
Parts:
- added JP4: JMP_5V, symbol Jumper:Jumper_2_Open
- added R31, R32: 10k, Resistor_SMD:R_0402_1005Metric, symbol Device:R
- J1: footprint Connector_PinSocket_2.54mm:PinSocket_2x20_P2.54mm_Vertical -> Connector_PinSocket_2.54mm:PinSocket_2x20_P2.54mm_Vertical_SMD
Connections:
- net GPIO36: no longer J1.37 (Pin_37)
- net GPIO37: no longer J1.38 (Pin_38)
- net GPIO38: no longer J1.39 (Pin_39)
- net GPIO39: no longer J1.40 (Pin_40)
- net GPIO8: now also R31.2
- net GPIO9: now also R32.2
- new net +3V3: R31.1, R32.1
- new net +5V: J1.37 (Pin_37), J1.38 (Pin_38), JP4.2 (B)
- new net GND: J1.39 (Pin_39), J1.40 (Pin_40)
- new net Power 5V/POWER_OUT: JP4.1 (A)
Other:
- sheet Power renamed Power 5V
- added sheet ESP32-C6 Wireless Co-Processor (esp32_c6_wireless_co_processor.kicad_sch)
- sheet Battery Management ports: added BATT_OUT; removed BATT_EN1, BATT_EN2, BATT_~{CHG}, BATT_~{PGOOD}
- sheet Power 5V ports: added IN, POWER_EN, POWER_IN, POWER_OUT, POWER_SCL, POWER_SDA; removed none
- sheet USB-C PD ports: added UCPD_FLIP, UCPD_GPIO, UCPD_INT, UCPD_SCL, UCPD_SDA; removed none
- moved on the sheet: H1, H2

Commit message: A
Connections:
- net BATT_OUT: now also J1.19 (Pin_19), J1.20 (Pin_20)
- net GPIO10: now also J1.9 (Pin_9); no longer J1.11 (Pin_11)
- net GPIO11: now also J1.10 (Pin_10); no longer J1.12 (Pin_12)
- net GPIO12: now also J1.11 (Pin_11); no longer J1.13 (Pin_13)
- net GPIO13: now also J1.12 (Pin_12); no longer J1.14 (Pin_14)
- net GPIO14: now also J1.13 (Pin_13); no longer J1.15 (Pin_15)
- net GPIO15: now also J1.14 (Pin_14); no longer J1.16 (Pin_16)
- net GPIO16: now also J1.15 (Pin_15); no longer J1.17 (Pin_17)
- net GPIO17: now also J1.16 (Pin_16); no longer J1.18 (Pin_18)
- net GPIO18: now also J1.17 (Pin_17); no longer J1.19 (Pin_19)
- net GPIO19: now also J1.18 (Pin_18); no longer J1.20 (Pin_20)
- net GPIO8: no longer J1.9 (Pin_9)
- net GPIO9: no longer J1.10 (Pin_10)
Other:
- sheet Power 5V ports: added none; removed IN
Changed lines of the file:
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@@
 		(color 0 0 0 0)
 	)
+	(junction
+		(at 220.98 74.93)
+		(diameter 0)
+		(color 0 0 0 0)
+	)
 	(no_connect
 		(at 257.81 149.86)
@@
 	)
 	(bus_entry
-		(at 215.9 69.85)
-		(size 2.54 2.54)
-		(stroke
-			(width 0)
-			(type default)
-		)
-	)
-	(bus_entry
 		(at 248.92 59.69)
 		(size -2.54 2.54)
@@
 	)
 	(bus_entry
-		(at 215.9 72.39)
-		(size 2.54 2.54)
-		(stroke
-			(width 0)
-			(type default)
-		)
-	)
-	(bus_entry
 		(at 248.92 39.37)
 		(size -2.54 2.54)
@@
 	(wire
 		(pts
-			(xy 218.44 72.39) (xy 226.06 72.39)
+			(xy 50.8 119.38) (xy 58.42 119.38)
 		)
 		(stroke
@@
 	(wire
 		(pts
+			(xy 220.98 72.39) (xy 226.06 72.39)
+		)
+		(stroke
+			(width 0)
+			(type default)
+		)
+	)
+	(wire
+		(pts
 			(xy 218.44 69.85) (xy 226.06 69.85)
 		)
@@
 	(wire
 		(pts
-			(xy 50.8 114.3) (xy 58.42 114.3)
-		)
-		(stroke
-			(width 0)
-			(type default)
-		)
-	)
-	(wire
-		(pts
 			(xy 111.76 121.92) (xy 124.46 121.92)
 		)
@@
 	(wire
 		(pts
+			(xy 220.98 72.39) (xy 220.98 74.93)
+		)
+		(stroke
+			(width 0)
+			(type default)
+		)
+	)
+	(wire
+		(pts
 			(xy 50.8 80.01) (xy 57.15 80.01)
 		)
@@
 	(wire
 		(pts
+			(xy 213.36 74.93) (xy 220.98 74.93)
+		)
+		(stroke
+			(width 0)
+			(type default)
+		)
+	)
+	(wire
+		(pts
 			(xy 254 64.77) (xy 254 67.31)
 		)
@@
 	(wire
 		(pts
-			(xy 218.44 74.93) (xy 226.06 74.93)
-		)
-		(stroke
-			(width 0)
-			(type default)
-		)
-	)
-	(wire
-		(pts
 			(xy 218.44 41.91) (xy 226.06 41.91)
 		)
@@
 	(wire
 		(pts
-			(xy 50.8 119.38) (xy 58.42 119.38)
+			(xy 238.76 74.93) (xy 246.38 74.93)
 		)
 		(stroke
@@
 	(wire
 		(pts
-			(xy 238.76 74.93) (xy 246.38 74.93)
+			(xy 144.78 44.45) (xy 147.32 44.45)
 		)
 		(stroke
@@
 	(wire
 		(pts
-			(xy 144.78 44.45) (xy 147.32 44.45)
+			(xy 111.76 129.54) (xy 124.46 129.54)
 		)
 		(stroke
@@
 	(wire
 		(pts
-			(xy 111.76 129.54) (xy 124.46 129.54)
+			(xy 220.98 74.93) (xy 226.06 74.93)
 		)
 		(stroke
@@
 	)
 	(label "BATT_OUT"
-		(at 58.42 114.3 0)
+		(at 58.42 119.38 0)
 		(effects
 			(font
@@
 		)
 	)
-	(label "GPIO37"
-		(at 238.76 85.09 0)
-		(effects
-			(font
-				(size 1.27 1.27)
-			)
-			(justify left bottom)
-		)
-	)
 	(label "GPIO8"
 		(at 58.42 127 0)
@@
 	)
 	(label "GPIO12"
-		(at 218.44 57.15 0)
+		(at 218.44 52.07 0)
 		(effects
 			(font
@@
 	)
 	(label "GPIO16"
-		(at 218.44 67.31 0)
+		(at 218.44 62.23 0)
 		(effects
 			(font
@@
 	)
 	(label "GPIO9"
-		(at 218.44 49.53 0)
-		(effects
-			(font
-				(size 1.27 1.27)
-			)
-			(justify left bottom)
-		)
-	)
-	(label "GPIO9"
 		(at 161.29 44.45 180)
 		(effects
@@
 		)
 	)
-	(label "GPIO9"
-		(at 58.42 124.46 0)
+	(label "BATT_OUT"
+		(at 213.36 74.93 180)
 		(effects
 			(font
 				(size 1.27 1.27)
 			)
-			(justify left bottom)
+			(justify right bottom)
 		)
 	)
-	(label "GPIO[0..39]"
-		(at 256.54 22.86 0)
+	(label "GPIO9"
+		(at 58.42 124.46 0)
 		(effects
 			(font
@@
 		)
 	)
-	(label "GPIO5"
-		(at 58.42 119.38 0)
+	(label "GPIO[0..39]"
+		(at 256.54 22.86 0)
 		(effects
 			(font
@@
 	)
 	(label "GPIO14"
-		(at 218.44 62.23 0)
+		(at 218.44 57.15 0)
 		(effects
 			(font
@@
 	)
 	(label "GPIO17"
-		(at 218.44 69.85 0)
+		(at 218.44 64.77 0)
 		(effects
 			(font
@@
 		)
 	)
-	(label "GPIO36"
-		(at 238.76 82.55 0)
-		(effects
-			(font
-				(size 1.27 1.27)
-			)
-			(justify left bottom)
-		)
-	)
 	(label "GPIO19"
 		(at 124.46 124.46 0)
@@
 	)
 	(label "GPIO15"
-		(at 218.44 64.77 0)
+		(at 218.44 59.69 0)
 		(effects
 			(font
@@
 		)
 	)
-	(label "GPIO39"
-		(at 238.76 90.17 0)
-		(effects
-			(font
-				(size 1.27 1.27)
-			)
-			(justify left bottom)
-		)
-	)
 	(label "GPIO11"
 		(at 124.46 116.84 0)
@@
 		)
 	)
-	(label "GPIO8"
-		(at 218.44 46.99 0)
-		(effects
-			(font
-				(size 1.27 1.27)
-			)
-			(justify left bottom)
-		)
-	)
 	(label "GPIO6"
 		(at 218.44 41.91 0)
@@
 	)
 	(label "GPIO11"
-		(at 218.44 54.61 0)
+		(at 218.44 49.53 0)
 		(effects
 			(font
@@
 	)
 	(label "GPIO10"
-		(at 218.44 52.07 0)
+		(at 218.44 46.99 0)
 		(effects
 			(font
@@
 	)
 	(label "GPIO18"
-		(at 218.44 72.39 0)
+		(at 218.44 67.31 0)
 		(effects
 			(font
@@
 		)
 	)
-	(label "GPIO38"
-		(at 238.76 87.63 0)
-		(effects
-			(font
-				(size 1.27 1.27)
-			)
-			(justify left bottom)
-		)
-	)
 	(label "GPIO9"
 		(at 118.11 30.48 0)
@@
 	)
 	(label "GPIO19"
-		(at 218.44 74.93 0)
+		(at 218.44 69.85 0)
 		(effects
 			(font
@@
 	)
 	(label "GPIO13"
-		(at 218.44 59.69 0)
+		(at 218.44 54.61 0)
 		(effects
 			(font
@@
 			)
 		)
-		(pin "IN" input
-			(at 50.8 114.3 0)
-			(effects
-				(font
-					(size 1.27 1.27)
-				)
-				(justify right)
-			)
-		)
