File: ControlCardRP/Hardware/Rev1/ControlCardRP/controller.kicad_sch (KiCad schematic)
At the start: 36 parts, among them J3 SWD, SW101 BOOT0, SW102 NRST, U101 W25Q128JVS, U102 RP2354B, U103 W25Q128JVS, Y1 12MHz

Commit message: A
Parts:
- added C121: 100n, Capacitor_SMD:C_0402_1005Metric, symbol Device:C
- added C21, C25: 10u, Capacitor_SMD:C_0603_1608Metric, symbol Device:C
- added D6, D7: LED, LED_SMD:LED_0603_1608Metric, symbol Device:LED
- added J9: Conn_01x03_Pin, Connector_PinHeader_1.27mm:PinHeader_1x03_P1.27mm_Vertical, symbol Connector:Conn_01x03_Pin
- added R109: 0R, Resistor_SMD:R_0402_1005Metric, symbol Device:R
- added R17, R18: 10k, Resistor_SMD:R_0402_1005Metric, symbol Device:R
- added U6: AZ1117-3.3, Package_TO_SOT_SMD:SOT-223-3_TabPin2, symbol Regulator_Linear:AZ1117-3.3
- C101: LCSC Part # (none) -> C23733
- C102, C103, C104, C105, C106, C107, C108, C109, C114, C115, C116, C117, C118: footprint Capacitor_SMD:C_0603_1608Metric -> Capacitor_SMD:C_0402_1005Metric; LCSC Part # (none) -> C1525
- C110, C111, C112, C113: footprint Capacitor_SMD:C_0603_1608Metric -> Capacitor_SMD:C_0402_1005Metric; LCSC Part # (none) -> C23733
- C119, C120: footprint Capacitor_SMD:C_0603_1608Metric -> Capacitor_SMD:C_0402_1005Metric; LCSC Part # (none) -> C1548
- L101: footprint Inductor_SMD:L_0805_2012Metric -> footprints:AOTA-B201610S3R3-101-T
- R101, R103, R104: footprint Resistor_SMD:R_0603_1608Metric -> Resistor_SMD:R_0402_1005Metric
- R102, R106, R107, R108: value 1k -> 10k; footprint Resistor_SMD:R_0603_1608Metric -> Resistor_SMD:R_0402_1005Metric; LCSC Part # (none) -> C25744
- R105: footprint Resistor_SMD:R_0603_1608Metric -> Resistor_SMD:R_0402_1005Metric; LCSC Part # (none) -> C17168
- U101: LCSC Part # (none) -> C97521
- U102: value RP2354B -> RP2350B; footprint Package_DFN_QFN:QFN-80-1EP_10x10mm_P0.4mm_EP3.4x3.4mm_ThermalVias -> Package_DFN_QFN:QFN-80-1EP_10x10mm_P0.4mm_EP3.4x3.4mm; symbol MCU_RaspberryPi:RP2354B -> MCU_RaspberryPi:RP2350B
Connections:
- net VREG_VIN is gone; now on net +3V3: U102.64 (VREG_VIN)
- net +3V3: now also C121.1, C25.1, R18.1, U6.2 (VO)
- net GND: now also C121.2, C21.2, C25.2, D6.1 (K), D7.1 (K), U6.1 (GND)
- net GPIO0: now also R109.2; no longer R107.2, U103.1 (~{CS})
- new net: R107.2, R109.1, U103.1 (~{CS})
- new net: C21.1, J9.2 (Pin_2), R17.1, U6.3 (VI)
- new net: D7.2 (A), R18.2
- new net: D6.2 (A), R17.2
- new net +5V: J9.3 (Pin_3)
- new net VBUS_UCPD: J9.1 (Pin_1)
Other:
- moved on the sheet: C118, R106, R107, R108, SW101, SW102, U103

Commit message: A
Parts:
- removed U101: W25Q128JVS, Package_SO:SOIC-8_5.3x5.3mm_P1.27mm, symbol Memory_Flash:W25Q128JVS
- added U7: W25Q128JVP, Package_SON:WSON-8-1EP_6x5mm_P1.27mm_EP3.4x4.3mm, symbol Memory_Flash:W25Q128JVP
Connections:
- net +3V3: now also U7.8 (VCC)
- net GND: now also U7.4 (GND), U7.9 (EP)
- net QSPI_SCLK: now also U7.6 (CLK)
- net QSPI_SD0: now also U7.5 (DI/IO_{0})
- net QSPI_SD1: now also U7.2 (DO/IO_{1})
- net QSPI_SD2: now also U7.3 (~{WP}/IO_{2})
- net QSPI_SD3: now also U7.7 (~{HOLD}/~{RESET}/IO_{3})
- net at R105.1: now also U7.1 (~{CS})
Changed lines of the file:
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@@
 	)
 	(junction
+		(at 40.64 132.08)
+		(diameter 0)
+		(color 0 0 0 0)
+	)
+	(junction
 		(at 172.72 25.4)
 		(diameter 0)
@@
 	(wire
 		(pts
-			(xy 76.2 147.32) (xy 78.74 147.32)
+			(xy 40.64 134.62) (xy 40.64 132.08)
 		)
 		(stroke
@@
 	(wire
 		(pts
-			(xy 156.21 186.69) (xy 156.21 185.42)
+			(xy 76.2 147.32) (xy 78.74 147.32)
 		)
 		(stroke
@@
 	(wire
 		(pts
-			(xy 25.4 22.86) (xy 25.4 25.4)
+			(xy 156.21 186.69) (xy 156.21 185.42)
 		)
 		(stroke
@@
 	(wire
 		(pts
-			(xy 50.8 121.92) (xy 78.74 121.92)
+			(xy 25.4 22.86) (xy 25.4 25.4)
 		)
 		(stroke
@@
 	(wire
 		(pts
-			(xy 129.54 99.06) (xy 138.43 99.06)
+			(xy 50.8 121.92) (xy 78.74 121.92)
 		)
 		(stroke
@@
 	(wire
 		(pts
-			(xy 40.64 129.54) (xy 40.64 132.08)
+			(xy 129.54 99.06) (xy 138.43 99.06)
 		)
 		(stroke
@@
 	(wire
 		(pts
+			(xy 38.1 129.54) (xy 38.1 132.08)
+		)
+		(stroke
+			(width 0)
+			(type default)
+		)
+	)
+	(wire
+		(pts
 			(xy 208.28 58.42) (xy 208.28 60.96)
 		)
@@
 	(wire
 		(pts
+			(xy 38.1 132.08) (xy 40.64 132.08)
+		)
+		(stroke
+			(width 0)
+			(type default)
+		)
+	)
+	(wire
+		(pts
 			(xy 25.4 45.72) (xy 25.4 48.26)
 		)
@@
 	(wire
 		(pts
+			(xy 40.64 129.54) (xy 40.64 132.08)
+		)
+		(stroke
+			(width 0)
+			(type default)
+		)
+	)
+	(wire
+		(pts
 			(xy 134.62 48.26) (xy 147.32 48.26)
 		)
@@
 	(symbol
 		(lib_id "power:GND")
-		(at 40.64 132.08 0)
+		(at 40.64 134.62 0)
 		(unit 1)
 		(body_style 1)
@@
 		(fields_autoplaced yes)
 		(property "Reference" "#PWR0113"
-			(at 40.64 138.43 0)
+			(at 40.64 140.97 0)
 			(hide yes)
 			(show_name no)
@@
 		)
 		(property "Value" "GND"
-			(at 40.64 137.16 0)
+			(at 40.64 139.7 0)
 			(show_name no)
 			(do_not_autoplace no)
@@
 		)
 		(property "Footprint" ""
-			(at 40.64 132.08 0)
+			(at 40.64 134.62 0)
 			(hide yes)
 			(show_name no)
@@
 		)
 		(property "Datasheet" ""
-			(at 40.64 132.08 0)
+			(at 40.64 134.62 0)
 			(hide yes)
 			(show_name no)
@@
 		)
 		(property "Description" "Power symbol creates a global label with name \"GND\" , ground"
-			(at 40.64 132.08 0)
+			(at 40.64 134.62 0)
 			(hide yes)
 			(show_name no)
@@
 	)
 	(symbol
+		(lib_id "Memory_Flash:W25Q128JVP")
+		(at 40.64 116.84 0)
+		(mirror y)
+		(unit 1)
+		(body_style 1)
+		(exclude_from_sim no)
+		(in_bom yes)
+		(on_board yes)
+		(in_pos_files yes)
+		(dnp no)
+		(fields_autoplaced yes)
+		(property "Reference" "U7"
+			(at 29.21 115.5699 0)
+			(show_name no)
+			(do_not_autoplace no)
+			(effects
+				(font
+					(size 1.27 1.27)
+				)
+				(justify left)
+			)
+		)
+		(property "Value" "W25Q128JVP"
+			(at 29.21 118.1099 0)
+			(show_name no)
+			(do_not_autoplace no)
+			(effects
+				(font
+					(size 1.27 1.27)
+				)
+				(justify left)
+			)
+		)
+		(property "Footprint" "Package_SON:WSON-8-1EP_6x5mm_P1.27mm_EP3.4x4.3mm"
+			(at 40.64 93.98 0)
+			(hide yes)
+			(show_name no)
+			(do_not_autoplace no)
+			(effects
+				(font
+					(size 1.27 1.27)
+				)
+			)
+		)
+		(property "Datasheet" "https://www.winbond.com/resource-files/w25q128jv_dtr%20revc%2003272018%20plus.pdf"
+			(at 40.64 91.44 0)
+			(hide yes)
+			(show_name no)
+			(do_not_autoplace no)
+			(effects
+				(font
+					(size 1.27 1.27)
+				)
+			)
+		)
+		(property "Description" "128Mbit / 16MiB Serial Flash Memory, Standard/Dual/Quad SPI, 2.7-3.6V, WSON-8"
+			(at 40.64 88.9 0)
+			(hide yes)
+			(show_name no)
+			(do_not_autoplace no)
+			(effects
+				(font
+					(size 1.27 1.27)
+				)
+			)
+		)
+		(pin "4"
+		)
+		(pin "5"
+		)
+		(pin "7"
+		)
+		(pin "2"
+		)
+		(pin "8"
+		)
+		(pin "1"
+		)
+		(pin "6"
+		)
+		(pin "3"
+		)
+		(pin "9"
+		)
+		(instances
+			(project "ControlCardRP"
+				(path "/a4806da1-c544-4ae5-b204-32c833e6ad2b/367b0da4-fb4c-4308-aa2b-30684a440207"
+					(reference "U7")
+					(unit 1)
+				)
+			)
+		)
+	)
+	(symbol
 		(lib_id "power:+5V")
 		(at 193.04 57.15 0)
@@
 					(unit 1)
 				)
-			)
-		)
-	)
-	(symbol
-		(lib_id "Memory_Flash:W25Q128JVS")
-		(at 40.64 116.84 0)
-		(mirror y)
-		(unit 1)
-		(body_style 1)
-		(exclude_from_sim no)
-		(in_bom yes)
-		(on_board yes)
-		(in_pos_files yes)
-		(dnp no)
-		(property "Reference" "U101"
-			(at 59.944 126.746 0)
-			(show_name no)
-			(do_not_autoplace no)
-			(effects
-				(font
-					(size 1.27 1.27)
-				)
-				(justify left)
-			)
-		)
-		(property "Value" "W25Q128JVS"
-			(at 59.944 129.286 0)
-			(show_name no)
-			(do_not_autoplace no)
-			(effects
-				(font
-					(size 1.27 1.27)
-				)
-				(justify left)
-			)
-		)
-		(property "Footprint" "Package_SO:SOIC-8_5.3x5.3mm_P1.27mm"
-			(at 40.64 93.98 0)
-			(hide yes)
-			(show_name no)
-			(do_not_autoplace no)
-			(effects
-				(font
-					(size 1.27 1.27)
-				)
-			)
-		)
-		(property "Datasheet" "https://www.winbond.com/resource-files/w25q128jv_dtr%20revc%2003272018%20plus.pdf"
-			(at 40.64 91.44 0)
-			(hide yes)
-			(show_name no)
-			(do_not_autoplace no)
-			(effects
-				(font
-					(size 1.27 1.27)
-				)
-			)
-		)
-		(property "Description" "128Mbit / 16MiB Serial Flash Memory, Standard/Dual/Quad SPI, 2.7-3.6V, SOIC-8"
-			(at 40.64 88.9 0)
-			(hide yes)
-			(show_name no)
-			(do_not_autoplace no)
-			(effects
-				(font
-					(size 1.27 1.27)
-				)
-			)
-		)
-		(property "LCSC Part #" "C97521"
-			(at 40.64 116.84 0)
-			(hide yes)
-			(show_name no)
-			(do_not_autoplace no)
-			(effects
-				(font
-					(size 1.27 1.27)
-				)
-			)
-		)
-		(property "KLC_S3.3" ""
-			(at 40.64 116.84 0)
-			(hide yes)
-			(show_name no)
-			(do_not_autoplace no)
-			(effects
-				(font
-					(size 1.27 1.27)
-				)
-			)
-		)
-		(property "KLC_S4.1" ""
-			(at 40.64 116.84 0)
-			(hide yes)
-			(show_name no)
-			(do_not_autoplace no)
-			(effects
-				(font
-					(size 1.27 1.27)
-				)
-			)
-		)
-		(property "KLC_S4.2_DVDD" ""
-			(at 40.64 116.84 0)
-			(hide yes)
-			(show_name no)
-			(do_not_autoplace no)
-			(effects
-				(font
-					(size 1.27 1.27)
-				)
-			)
-		)
-		(property "KLC_S4.2_VCC" ""
-			(at 40.64 116.84 0)
-			(hide yes)
-			(show_name no)
-			(do_not_autoplace no)
-			(effects
-				(font
-					(size 1.27 1.27)
-				)
-			)
-		)
-		(property "KLC_S4.2_VREG_LX" ""
-			(at 40.64 116.84 0)
-			(hide yes)
-			(show_name no)
-			(do_not_autoplace no)
-			(effects
-				(font
-					(size 1.27 1.27)
-				)
-			)
-		)
-		(property "KLC_S4.4" ""
-			(at 40.64 116.84 0)
-			(hide yes)
-			(show_name no)
-			(do_not_autoplace no)
-			(effects
-				(font
-					(size 1.27 1.27)
-				)
-			)
-		)
-		(pin "3"
-		)
-		(pin "7"
-		)
-		(pin "1"
-		)
-		(pin "2"
-		)
-		(pin "5"
-		)
-		(pin "8"
-		)
-		(pin "4"
-		)
-		(pin "6"
-		)
-		(instances
-			(project "ControlCardRP"
-				(path "/a4806da1-c544-4ae5-b204-32c833e6ad2b/367b0da4-fb4c-4308-aa2b-30684a440207"
-					(reference "U101")
-					(unit 1)
-				)
