File: ControlCardRP/Hardware/Rev1/ControlCardRP/controller.kicad_sch (KiCad schematic)
At the start: 46 parts, among them J3 SWD, J9 Conn_01x03_Pin, SW101 BOOT0, SW102 NRST, U102 RP2350B, U103 W25Q128JVS, U6 AZ1117-3.3, U7 W25Q128JVS, Y1 12MHz

Commit message: A
Parts:
- C21, C25: LCSC Part # C440198 -> C96446
Changed lines of the file:
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@@
 			)
 		)
-		(property "LCSC Part #" "C440198"
+		(property "LCSC Part #" "C96446"
 			(at 224.79 69.85 0)
 			(hide yes)
@@
 			)
 		)
-		(property "LCSC Part #" "C440198"
+		(property "LCSC Part #" "C96446"
 			(at 255.27 69.85 0)
 			(hide yes)

Commit message: A
Parts:
- C101: footprint Capacitor_SMD:C_0603_1608Metric -> Capacitor_SMD:C_0402_1005Metric
- R101: LCSC Part # (none) -> C25105
- R103, R104: footprint Resistor_SMD:R_0402_1005Metric -> Resistor_SMD:R_0603_1608Metric; LCSC Part # (none) -> C25190
Changed lines of the file:
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@@
 			)
 		)
-		(property "Footprint" "Capacitor_SMD:C_0603_1608Metric"
+		(property "Footprint" "Capacitor_SMD:C_0402_1005Metric"
 			(at 110.1852 35.56 0)
 			(hide yes)
@@
 			)
 		)
-		(property "Footprint" "Resistor_SMD:R_0402_1005Metric"
+		(property "Footprint" "Resistor_SMD:R_0603_1608Metric"
 			(at 62.23 100.838 90)
 			(hide yes)
@@
 			)
 		)
-		(property "LCSC Part #" ""
+		(property "LCSC Part #" "C25190"
 			(at 62.23 99.06 90)
 			(hide yes)
@@
 			)
 		)
-		(property "Footprint" "Resistor_SMD:R_0402_1005Metric"
+		(property "Footprint" "Resistor_SMD:R_0603_1608Metric"
 			(at 62.23 103.378 90)
 			(hide yes)
@@
 			)
 		)
-		(property "LCSC Part #" ""
+		(property "LCSC Part #" "C25190"
 			(at 62.23 101.6 90)
 			(hide yes)
@@
 			)
 		)
-		(property "LCSC Part #" ""
+		(property "LCSC Part #" "C25105"
 			(at 52.07 25.4 90)
 			(hide yes)
