File: ControlCardRP/Hardware/Rev1/ControlCardRP/esp32_s3_wireless_co_processor.kicad_sch (KiCad schematic)
At the start: 1 part, among them U5 ESP32-S3

Commit message: A
Parts:
- removed U5: ESP32-S3, Package_DFN_QFN:QFN-56-1EP_7x7mm_P0.4mm_EP4x4mm, symbol MCU_Espressif:ESP32-S3
- added U5: ESP32-C3, Package_DFN_QFN:QFN-32-1EP_5x5mm_P0.5mm_EP3.7x3.7mm, symbol MCU_Espressif:ESP32-C3
Connections:
- new net: U5.2 (VDD3P3), U5.3 (VDD3P3)
- new net: U5.31 (VDDA), U5.32 (VDDA)
Changed lines of the file:
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@@
 	(paper "A4")
 	(symbol
-		(lib_id "MCU_Espressif:ESP32-S3")
-		(at 67.31 67.31 0)
+		(lib_id "MCU_Espressif:ESP32-C3")
+		(at 137.16 99.06 0)
 		(unit 1)
 		(body_style 1)
@@
 		(fields_autoplaced yes)
 		(property "Reference" "U5"
-			(at 69.4533 105.41 0)
+			(at 139.3033 124.46 0)
 			(show_name no)
 			(do_not_autoplace no)
@@
 			)
 		)
-		(property "Value" "ESP32-S3"
-			(at 69.4533 107.95 0)
+		(property "Value" "ESP32-C3"
+			(at 139.3033 127 0)
 			(show_name no)
 			(do_not_autoplace no)
@@
 			)
 		)
-		(property "Footprint" "Package_DFN_QFN:QFN-56-1EP_7x7mm_P0.4mm_EP4x4mm"
-			(at 67.31 115.57 0)
+		(property "Footprint" "Package_DFN_QFN:QFN-32-1EP_5x5mm_P0.5mm_EP3.7x3.7mm"
+			(at 137.668 99.06 0)
 			(hide yes)
 			(show_name no)
@@
 			)
 		)
-		(property "Datasheet" "https://www.espressif.com/sites/default/files/documentation/esp32-s3_datasheet_en.pdf"
-			(at 67.31 67.31 0)
+		(property "Datasheet" "https://www.espressif.com/sites/default/files/documentation/esp32-c3_datasheet_en.pdf"
+			(at 137.668 99.06 0)
 			(hide yes)
 			(show_name no)
@@
 			)
 		)
-		(property "Description" "Microcontroller, Wi-Fi 802.11b/g/n, Bluetooth, 32bit"
-			(at 67.31 67.31 0)
+		(property "Description" "RF Module, ESP32 SoC, RISC-V, WiFi 802.11b/n/g, Bluetooth LE 5, QFN32"
+			(at 137.668 99.06 0)
 			(hide yes)
 			(show_name no)
@@
 			)
 		)
-		(pin "50"
+		(pin "20"
 		)
-		(pin "54"
+		(pin "14"
 		)
-		(pin "39"
+		(pin "24"
 		)
-		(pin "40"
+		(pin "26"
 		)
-		(pin "43"
+		(pin "13"
 		)
-		(pin "46"
+		(pin "29"
 		)
-		(pin "41"
+		(pin "9"
 		)
-		(pin "44"
+		(pin "17"
 		)
-		(pin "47"
+		(pin "12"
 		)
-		(pin "48"
+		(pin "5"
 		)
-		(pin "57"
+		(pin "10"
 		)
-		(pin "55"
+		(pin "7"
 		)
-		(pin "49"
+		(pin "1"
 		)
-		(pin "52"
+		(pin "2"
 		)
-		(pin "42"
+		(pin "3"
 		)
-		(pin "53"
+		(pin "11"
 		)
 		(pin "8"
 		)
-		(pin "16"
-		)
 		(pin "18"
 		)
-		(pin "6"
+		(pin "4"
 		)
-		(pin "7"
+		(pin "15"
 		)
-		(pin "14"
-		)
-		(pin "25"
-		)
-		(pin "13"
+		(pin "16"
 		)
 		(pin "19"
 		)
-		(pin "51"
-		)
-		(pin "2"
-		)
-		(pin "24"
-		)
-		(pin "3"
-		)
-		(pin "5"
-		)
-		(pin "12"
-		)
-		(pin "56"
-		)
-		(pin "10"
-		)
-		(pin "15"
-		)
-		(pin "36"
-		)
-		(pin "1"
-		)
-		(pin "9"
-		)
-		(pin "45"
-		)
-		(pin "4"
-		)
-		(pin "11"
-		)
-		(pin "17"
-		)
-		(pin "20"
+		(pin "6"
 		)
 		(pin "21"
@@
 		(pin "23"
 		)
-		(pin "26"
+		(pin "25"
+		)
+		(pin "27"
 		)
 		(pin "28"
 		)
-		(pin "29"
+		(pin "30"
 		)
-		(pin "30"
+		(pin "32"
 		)
 		(pin "31"
 		)
-		(pin "32"
-		)
 		(pin "33"
 		)
-		(pin "37"
-		)
-		(pin "38"
-		)
-		(pin "27"
-		)
-		(pin "34"
-		)
-		(pin "35"
-		)
 		(instances
