File: ControlCardRP/Hardware/Rev1/ControlCardRP/Production/ControlCardRP_panelized.kicad_pcb (KiCad board)
At the start: 4 copper layers, 53.5 x 49.5 mm, 153 parts, among them J1 Conn_02x20_Top_Bottom, J2 USB_C_Receptacle_USB2.0_16P, J3 SWD, J4 JST_PK BATTERY, J5 PIN_HEADER BATTERY, J8 ESP_IO, J9 Conn_01x03_Pin, Q1 NMOS, Q2 NMOS, SW1 SW_SPST, SW101 BOOT0, SW102 NRST, SW103 NRST, SW104 NRST, U1 AP33772SDKZ-xx-FA02, U102 RP2350B, U103 W25Q128JVS, U2 BQ24075RGT, U3 BQ27427YZFR, U4 MP28167GQ-A-P, U5 ESP32-C6-MINI-1, U6 AZ1117-3.3, U7 W25Q128JVP, Y1 12MHz

Commit message: A
Parts:
- added ?: , Fiducial_1.5mm_Mask3mm, F.Cu at (118.5, 112.0)
- added ?: , Fiducial_1mm_Mask3mm, F.Cu at (177.0, 66.5)
- added ?: , Fiducial_1mm_Mask3mm, F.Cu at (118.5, 66.5)
- added ?: , Fiducial_1mm_Mask3mm, B.Cu at (118.5, 66.5)
- added ?: , Fiducial_1.5mm_Mask3mm, B.Cu at (118.5, 112.0)
- added ?: , Fiducial_1mm_Mask3mm, B.Cu at (177.0, 66.5)
- U5: footprint footprints:ESP32-C6-MINI-1 -> RF_Module:ESP32-C6-MINI-1
Other:
- board size 53.5 x 49.5 mm -> 68.2 x 63.2 mm
- board text added: "Panelized"
- board text added: "ROUTE OUT"
- board text added: "V-SCORE"
