File: ControlCardRP/Hardware/Rev1/ControlCardRP/_restore_backup_2026-08-10T23-14-51-235/ControlCardRP.kicad_sch (KiCad schematic)
At the start: 7 parts, among them J1 Conn_02x20_Top_Bottom, J10 MAIN_POWER

Commit message: A
Parts:
- removed J10: MAIN_POWER, Connector_PinHeader_2.54mm:PinHeader_1x02_P2.54mm_Vertical, symbol Connector_Generic:Conn_01x02
- removed R66: 10k, Resistor_SMD:R_0402_1005Metric, symbol Device:R
- added JP4: JMP_5V, symbol Jumper:Jumper_2_Open
Connections:
- net GPIO41 is gone; now on net GPIO2: J1.3 (Pin_3)
- net GPIO42 is gone; now on net GPIO5: J1.6 (Pin_6)
- net GPIO43 is gone; now on net GPIO6: J1.7 (Pin_7)
- net GPIO44 is gone; now on net GPIO7: J1.8 (Pin_8)
- net +5V: now also JP4.2 (B)
- net GPIO19: now also J1.18 (Pin_18)
- net GPIO34: now also J1.35 (Pin_35); no longer J1.17 (Pin_17)
- net GPIO35: now also J1.36 (Pin_36); no longer J1.18 (Pin_18)
- net GPIO40 renamed GPIO0
- removed net POWER_AUX: J1.35 (Pin_35), J1.36 (Pin_36)
- new net GPIO18: J1.17 (Pin_17)
- new net Power 5V/POWER_OUT: JP4.1 (A)
Other:
- removed sheet Power AUX
- sheet Controller ports: added GPIO[0..39]; removed GPIO[0..47]
- sheet Power 5V ports: added none; removed POWER_ALT
