File: ControlCardRP/Hardware/Rev1/ControlCardRP/_restore_backup_2026-08-10T23-14-51-235/battery_management.kicad_sch (KiCad schematic)
At the start: 29 parts, among them J4 JST_PK BATTERY, J5 PIN_HEADER BATTERY, SW1 SW_SPDT, U2 BQ24075RGT, U3 BQ27427YZFR

Commit message: A
Parts:
- SW1: value SW_SPDT -> SW_SPST; symbol Switch:SW_SPDT -> Switch:SW_SPST
Connections:
- net BATT_OUT: now also SW1.2 (B); no longer SW1.1 (A)
- net GND: now also J4.2 (Pin_2); no longer J4.1 (Pin_1), SW1.3 (C)
- net SYSOFF: now also SW1.1 (A); no longer SW1.2 (B)
- net at C8.1, J5.1 (Pin_1), U3.C3 (BAT): now also J4.1 (Pin_1); no longer J4.2 (Pin_2)
Other:
- moved on the sheet: J4
Changed lines of the file:
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@@
 	(wire
 		(pts
-			(xy 54.61 78.74) (xy 54.61 76.2)
-		)
-		(stroke
-			(width 0)
-			(type default)
-		)
-	)
-	(wire
-		(pts
 			(xy 194.31 92.71) (xy 194.31 77.47)
 		)
@@
 	(wire
 		(pts
-			(xy 52.07 71.12) (xy 54.61 71.12)
+			(xy 52.07 73.66) (xy 54.61 73.66)
 		)
 		(stroke
@@
 	(wire
 		(pts
-			(xy 54.61 76.2) (xy 52.07 76.2)
-		)
-		(stroke
-			(width 0)
-			(type default)
-		)
-	)
-	(wire
-		(pts
 			(xy 153.67 72.39) (xy 151.13 72.39)
 		)
@@
 	)
 	(label "OUT"
-		(at 54.61 71.12 0)
+		(at 54.61 73.66 0)
 		(effects
 			(font
@@
 	)
 	(symbol
-		(lib_id "Switch:SW_SPDT")
+		(lib_id "Switch:SW_SPST")
 		(at 46.99 73.66 0)
 		(unit 1)
@@
 		(fields_autoplaced yes)
 		(property "Reference" "SW1"
-			(at 46.99 64.77 0)
+			(at 46.99 67.31 0)
 			(show_name no)
 			(do_not_autoplace no)
@@
 			)
 		)
-		(property "Value" "SW_SPDT"
-			(at 46.99 67.31 0)
+		(property "Value" "SW_SPST"
+			(at 46.99 69.85 0)
 			(show_name no)
 			(do_not_autoplace no)
@@
 		)
 		(property "Datasheet" ""
-			(at 46.99 81.28 0)
+			(at 46.99 73.66 0)
 			(hide yes)
 			(show_name no)
@@
 			)
 		)
-		(property "Description" "Switch, single pole double throw"
+		(property "Description" "Single Pole Single Throw (SPST) switch"
 			(at 46.99 73.66 0)
 			(hide yes)
@@
 		(pin "1"
 		)
-		(pin "3"
-		)
 		(instances
 			(project "ControlCardRP"
@@
 	(symbol
 		(lib_id "Connector:Conn_01x02_Socket")
-		(at 186.69 95.25 180)
+		(at 186.69 92.71 0)
+		(mirror y)
 		(unit 1)
 		(body_style 1)
@@
 		(dnp no)
 		(property "Reference" "J4"
-			(at 184.15 87.376 0)
+			(at 184.658 88.9 0)
 			(show_name no)
 			(do_not_autoplace no)
@@
 		)
 		(property "Value" "JST_PK BATTERY"
-			(at 184.912 90.17 0)
+			(at 184.912 97.79 0)
 			(show_name no)
 			(do_not_autoplace no)
@@
 		)
 		(property "Footprint" "Connector_JST:JST_PH_S2B-PH-K_1x02_P2.00mm_Horizontal"
-			(at 186.69 95.25 0)
+			(at 186.69 92.71 0)
 			(hide yes)
 			(show_name no)
@@
 		)
 		(property "Datasheet" ""
-			(at 186.69 95.25 0)
+			(at 186.69 92.71 0)
 			(hide yes)
 			(show_name no)
@@
 		)
 		(property "Description" "Generic connector, single row, 01x02, script generated"
-			(at 186.69 95.25 0)
+			(at 186.69 92.71 0)
 			(hide yes)
 			(show_name no)
@@
 		)
 		(property "LCSC Part #" ""
-			(at 186.69 95.25 0)
+			(at 186.69 92.71 0)
 			(hide yes)
 			(show_name no)
@@
 		)
 		(property "KLC_S3.3" ""
-			(at 186.69 95.25 0)
+			(at 186.69 92.71 0)
 			(hide yes)
 			(show_name no)
@@
 		)
 		(property "KLC_S4.1" ""
-			(at 186.69 95.25 0)
+			(at 186.69 92.71 0)
 			(hide yes)
 			(show_name no)
@@
 		)
 		(property "KLC_S4.2_DVDD" ""
-			(at 186.69 95.25 0)
+			(at 186.69 92.71 0)
 			(hide yes)
 			(show_name no)
@@
 		)
 		(property "KLC_S4.2_VCC" ""
-			(at 186.69 95.25 0)
+			(at 186.69 92.71 0)
 			(hide yes)
 			(show_name no)
@@
 		)
 		(property "KLC_S4.2_VREG_LX" ""
-			(at 186.69 95.25 0)
+			(at 186.69 92.71 0)
 			(hide yes)
 			(show_name no)
@@
 		)
 		(property "KLC_S4.4" ""
-			(at 186.69 95.25 0)
+			(at 186.69 92.71 0)
 			(hide yes)
 			(show_name no)
@@
 					(unit 1)
 				)
-			)
-		)
-	)
-	(symbol
-		(lib_id "power:GND")
-		(at 54.61 78.74 0)
-		(unit 1)
-		(body_style 1)
-		(exclude_from_sim no)
-		(in_bom yes)
-		(on_board yes)
-		(in_pos_files yes)
-		(dnp no)
-		(fields_autoplaced yes)
-		(property "Reference" "#PWR056"
-			(at 54.61 85.09 0)
-			(hide yes)
-			(show_name no)
-			(do_not_autoplace no)
-			(effects
-				(font
-					(size 1.27 1.27)
-				)
-			)
-		)
-		(property "Value" "GND"
-			(at 54.61 83.82 0)
-			(show_name no)
-			(do_not_autoplace no)
-			(effects
-				(font
-					(size 1.27 1.27)
-				)
-			)
-		)
-		(property "Footprint" ""
-			(at 54.61 78.74 0)
-			(hide yes)
-			(show_name no)
-			(do_not_autoplace no)
-			(effects
-				(font
-					(size 1.27 1.27)
-				)
-			)
-		)
-		(property "Datasheet" ""
-			(at 54.61 78.74 0)
-			(hide yes)
-			(show_name no)
-			(do_not_autoplace no)
-			(effects
-				(font
-					(size 1.27 1.27)
-				)
-			)
-		)
-		(property "Description" "Power symbol creates a global label with name \"GND\" , ground"
-			(at 54.61 78.74 0)
-			(hide yes)
-			(show_name no)
-			(do_not_autoplace no)
-			(effects
-				(font
-					(size 1.27 1.27)
-				)
-			)
-		)
-		(pin "1"
-		)
-		(instances
-			(project "ControlCardRP"
-				(path "/a4806da1-c544-4ae5-b204-32c833e6ad2b/632eec67-69c0-4c64-a789-34cbb910d8dd"
-					(reference "#PWR056")
-					(unit 1)
-				)
