File: ControlCardRP/Hardware/Rev1/ControlCardRP/_restore_backup_2026-08-10T23-14-51-235/controller.kicad_sch (KiCad schematic)
At the start: 46 parts, among them J3 SWD, J9 Conn_01x03_Pin, SW101 BOOT0, SW102 NRST, U102 RP2350B, U103 W25Q128JVS, U6 AZ1117-3.3, U7 W25Q128JVS, Y1 12MHz

Commit message: A
Parts:
- U6: footprint Package_TO_SOT_SMD:SOT-89-3 -> Package_TO_SOT_SMD:SOT-223-3_TabPin2
- U7: value W25Q128JVS -> W25Q128JVP; footprint Package_SO:SOIC-8_5.3x5.3mm_P1.27mm -> Package_SON:WSON-8-1EP_6x5mm_P1.27mm_EP3.4x4.3mm; symbol Memory_Flash:W25Q128JVS -> Memory_Flash:W25Q128JVP
Connections:
- net GND: now also U7.9 (EP)
- net GPIO40 renamed GPIO40/ADC0
- net GPIO41 renamed GPIO41/ADC1
- net GPIO42 renamed GPIO42/ADC2
- net GPIO43 renamed GPIO43/ADC3
- net GPIO44 renamed GPIO44/ADC4
- net GPIO45 renamed GPIO45/ADC5
- net GPIO46 renamed GPIO46/ADC6
- net GPIO47 renamed GPIO47/ADC7
- no-connect marks 4 -> 0
Other:
- moved on the sheet: C118, R107, R109, U103
