File: ControlCardRP/Hardware/Rev1/ControlCardRP/_restore_backup_2026-08-10T23-14-51-235/esp32_c6_wireless_co_processor.kicad_sch (KiCad schematic)
At the start: 22 parts, among them J6 ESP_PROG_UART, J7 ESP_PROG_JTAG, J8 ESP_IO, SW103 NRST, SW104 NRST, U5 ESP32-C6-MINI-1

Commit message: A
Parts:
- U5: footprint footprints:ESP32-C6-MINI-1 -> RF_Module:ESP32-C6-MINI-1
Changed lines of the file:
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@@
 			)
 		)
-		(property "Footprint" "footprints:ESP32-C6-MINI-1"
+		(property "Footprint" "RF_Module:ESP32-C6-MINI-1"
 			(at 148.59 114.3 0)
 			(hide yes)
