File: ControlCardRP/Hardware/Rev1/ControlCardRP/_restore_backup_2026-08-10T23-14-51-235/power.kicad_sch (KiCad schematic)
At the start: 26 parts, among them U4 MP28167GQ-A-P

Commit message: A
Parts:
- R26, R27, R29: now not fitted
Changed lines of the file:
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@@
 					(unit 1)
 				)
-				(path "/a4806da1-c544-4ae5-b204-32c833e6ad2b/1569a62d-a1a0-464a-8dcd-6a4c810cd1dd"
-					(reference "#PWR060")
-					(unit 1)
-				)
 			)
 		)
@@
 					(unit 1)
 				)
-				(path "/a4806da1-c544-4ae5-b204-32c833e6ad2b/1569a62d-a1a0-464a-8dcd-6a4c810cd1dd"
-					(reference "C27")
-					(unit 1)
-				)
 			)
 		)
@@
 					(unit 1)
 				)
-				(path "/a4806da1-c544-4ae5-b204-32c833e6ad2b/1569a62d-a1a0-464a-8dcd-6a4c810cd1dd"
-					(reference "C36")
-					(unit 1)
-				)
 			)
 		)
@@
 					(unit 1)
 				)
-				(path "/a4806da1-c544-4ae5-b204-32c833e6ad2b/1569a62d-a1a0-464a-8dcd-6a4c810cd1dd"
-					(reference "R60")
-					(unit 1)
-				)
 			)
 		)
@@
 					(unit 1)
 				)
-				(path "/a4806da1-c544-4ae5-b204-32c833e6ad2b/1569a62d-a1a0-464a-8dcd-6a4c810cd1dd"
-					(reference "#PWR063")
-					(unit 1)
-				)
 			)
 		)
@@
 					(unit 1)
 				)
-				(path "/a4806da1-c544-4ae5-b204-32c833e6ad2b/1569a62d-a1a0-464a-8dcd-6a4c810cd1dd"
-					(reference "C26")
-					(unit 1)
-				)
 			)
 		)
@@
 					(unit 1)
 				)
-				(path "/a4806da1-c544-4ae5-b204-32c833e6ad2b/1569a62d-a1a0-464a-8dcd-6a4c810cd1dd"
-					(reference "C32")
-					(unit 1)
-				)
 			)
 		)
@@
 		(on_board yes)
 		(in_pos_files yes)
-		(dnp no)
+		(dnp yes)
 		(fields_autoplaced yes)
 		(property "Reference" "#PWR029"
@@
 					(unit 1)
 				)
-				(path "/a4806da1-c544-4ae5-b204-32c833e6ad2b/1569a62d-a1a0-464a-8dcd-6a4c810cd1dd"
-					(reference "#PWR065")
-					(unit 1)
-				)
 			)
 		)
@@
 					(unit 1)
 				)
-				(path "/a4806da1-c544-4ae5-b204-32c833e6ad2b/1569a62d-a1a0-464a-8dcd-6a4c810cd1dd"
-					(reference "R52")
-					(unit 1)
-				)
 			)
 		)
@@
 					(unit 1)
 				)
-				(path "/a4806da1-c544-4ae5-b204-32c833e6ad2b/1569a62d-a1a0-464a-8dcd-6a4c810cd1dd"
-					(reference "#PWR064")
-					(unit 1)
-				)
 			)
 		)
@@
 					(unit 1)
 				)
-				(path "/a4806da1-c544-4ae5-b204-32c833e6ad2b/1569a62d-a1a0-464a-8dcd-6a4c810cd1dd"
-					(reference "R57")
-					(unit 1)
-				)
 			)
 		)
@@
 					(unit 1)
 				)
-				(path "/a4806da1-c544-4ae5-b204-32c833e6ad2b/1569a62d-a1a0-464a-8dcd-6a4c810cd1dd"
-					(reference "R65")
-					(unit 1)
-				)
 			)
 		)
@@
 		(on_board yes)
 		(in_pos_files yes)
-		(dnp no)
+		(dnp yes)
 		(fields_autoplaced yes)
 		(property "Reference" "R27"
@@
 					(unit 1)
 				)
-				(path "/a4806da1-c544-4ae5-b204-32c833e6ad2b/1569a62d-a1a0-464a-8dcd-6a4c810cd1dd"
-					(reference "R62")
-					(unit 1)
-				)
 			)
 		)
@@
 					(unit 1)
 				)
-				(path "/a4806da1-c544-4ae5-b204-32c833e6ad2b/1569a62d-a1a0-464a-8dcd-6a4c810cd1dd"
-					(reference "C29")
-					(unit 1)
-				)
 			)
 		)
@@
 		(on_board yes)
 		(in_pos_files yes)
-		(dnp no)
+		(dnp yes)
 		(fields_autoplaced yes)
 		(property "Reference" "R26"
@@
 					(unit 1)
 				)
-				(path "/a4806da1-c544-4ae5-b204-32c833e6ad2b/1569a62d-a1a0-464a-8dcd-6a4c810cd1dd"
-					(reference "R61")
-					(unit 1)
-				)
 			)
 		)
@@
 					(unit 1)
 				)
-				(path "/a4806da1-c544-4ae5-b204-32c833e6ad2b/1569a62d-a1a0-464a-8dcd-6a4c810cd1dd"
-					(reference "L2")
-					(unit 1)
-				)
 			)
 		)
@@
 					(unit 1)
 				)
-				(path "/a4806da1-c544-4ae5-b204-32c833e6ad2b/1569a62d-a1a0-464a-8dcd-6a4c810cd1dd"
-					(reference "#PWR067")
-					(unit 1)
-				)
 			)
 		)
@@
 					(unit 1)
 				)
-				(path "/a4806da1-c544-4ae5-b204-32c833e6ad2b/1569a62d-a1a0-464a-8dcd-6a4c810cd1dd"
-					(reference "D12")
-					(unit 1)
-				)
 			)
 		)
@@
 					(unit 1)
 				)
-				(path "/a4806da1-c544-4ae5-b204-32c833e6ad2b/1569a62d-a1a0-464a-8dcd-6a4c810cd1dd"
-					(reference "C30")
-					(unit 1)
-				)
 			)
 		)
@@
 					(unit 1)
 				)
-				(path "/a4806da1-c544-4ae5-b204-32c833e6ad2b/1569a62d-a1a0-464a-8dcd-6a4c810cd1dd"
-					(reference "C33")
-					(unit 1)
-				)
 			)
 		)
@@
 					(unit 1)
 				)
-				(path "/a4806da1-c544-4ae5-b204-32c833e6ad2b/1569a62d-a1a0-464a-8dcd-6a4c810cd1dd"
-					(reference "R58")
-					(unit 1)
-				)
 			)
 		)
@@
 					(unit 1)
 				)
-				(path "/a4806da1-c544-4ae5-b204-32c833e6ad2b/1569a62d-a1a0-464a-8dcd-6a4c810cd1dd"
-					(reference "C34")
-					(unit 1)
-				)
 			)
 		)
@@
 					(unit 1)
 				)
-				(path "/a4806da1-c544-4ae5-b204-32c833e6ad2b/1569a62d-a1a0-464a-8dcd-6a4c810cd1dd"
-					(reference "C35")
-					(unit 1)
-				)
 			)
 		)
@@
 					(unit 1)
 				)
-				(path "/a4806da1-c544-4ae5-b204-32c833e6ad2b/1569a62d-a1a0-464a-8dcd-6a4c810cd1dd"
-					(reference "R64")
-					(unit 1)
-				)
 			)
 		)
@@
 					(unit 1)
 				)
-				(path "/a4806da1-c544-4ae5-b204-32c833e6ad2b/1569a62d-a1a0-464a-8dcd-6a4c810cd1dd"
-					(reference "R59")
-					(unit 1)
-				)
 			)
 		)
@@
 		(on_board yes)
 		(in_pos_files yes)
-		(dnp no)
+		(dnp yes)
 		(fields_autoplaced yes)
 		(property "Reference" "R29"
@@
 					(unit 1)
 				)
-				(path "/a4806da1-c544-4ae5-b204-32c833e6ad2b/1569a62d-a1a0-464a-8dcd-6a4c810cd1dd"
-					(reference "R63")
-					(unit 1)
-				)
 			)
 		)
@@
 					(unit 1)
 				)
-				(path "/a4806da1-c544-4ae5-b204-32c833e6ad2b/1569a62d-a1a0-464a-8dcd-6a4c810cd1dd"
-					(reference "C31")
-					(unit 1)
-				)
 			)
 		)
@@
 					(unit 1)
 				)
-				(path "/a4806da1-c544-4ae5-b204-32c833e6ad2b/1569a62d-a1a0-464a-8dcd-6a4c810cd1dd"
-					(reference "#PWR061")
-					(unit 1)
-				)
 			)
 		)
@@
 					(unit 1)
 				)
-				(path "/a4806da1-c544-4ae5-b204-32c833e6ad2b/1569a62d-a1a0-464a-8dcd-6a4c810cd1dd"
-					(reference "#PWR058")
-					(unit 1)
-				)
 			)
 		)
@@
 					(unit 1)
 				)
-				(path "/a4806da1-c544-4ae5-b204-32c833e6ad2b/1569a62d-a1a0-464a-8dcd-6a4c810cd1dd"
-					(reference "R53")
-					(unit 1)
-				)
 			)
 		)
@@
 					(unit 1)
 				)
-				(path "/a4806da1-c544-4ae5-b204-32c833e6ad2b/1569a62d-a1a0-464a-8dcd-6a4c810cd1dd"
-					(reference "#PWR068")
-					(unit 1)
-				)
 			)
 		)
@@
 					(unit 1)
 				)
-				(path "/a4806da1-c544-4ae5-b204-32c833e6ad2b/1569a62d-a1a0-464a-8dcd-6a4c810cd1dd"
-					(reference "R56")
-					(unit 1)
-				)
 			)
 		)
@@
 					(unit 1)
 				)
-				(path "/a4806da1-c544-4ae5-b204-32c833e6ad2b/1569a62d-a1a0-464a-8dcd-6a4c810cd1dd"
-					(reference "#PWR062")
-					(unit 1)
-				)
 			)
 		)
@@
 					(unit 1)
 				)
-				(path "/a4806da1-c544-4ae5-b204-32c833e6ad2b/1569a62d-a1a0-464a-8dcd-6a4c810cd1dd"
-					(reference "D9")
-					(unit 1)
-				)
 			)
 		)
@@
 					(unit 1)
 				)
-				(path "/a4806da1-c544-4ae5-b204-32c833e6ad2b/1569a62d-a1a0-464a-8dcd-6a4c810cd1dd"
-					(reference "#PWR066")
-					(unit 1)
-				)
 			)
 		)
@@
 					(unit 1)
 				)
-				(path "/a4806da1-c544-4ae5-b204-32c833e6ad2b/1569a62d-a1a0-464a-8dcd-6a4c810cd1dd"
-					(reference "U8")
-					(unit 1)
-				)
