File: ControlCardRP/Hardware/Rev1/ControlCardRP/_restore_backup_2026-08-10T23-14-51-235/usb_c_pd.kicad_sch (KiCad schematic)
At the start: 27 parts, among them J2 USB_C_Receptacle_USB2.0_16P, Q1 NMOS, Q2 NMOS, U1 AP33772SDKZ-xx-FA02

Commit message: A
Connections:
- net FLIP: no longer R44.2, U1.6 (FLIP)
- new net: R44.2, U1.6 (FLIP)
Changed lines of the file:
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@@
-		)
-	)
-	(label "FLIP"
-		(at 143.51 91.44 0)
-		(effects
-			(font
-				(size 1.27 1.27)
-			)
-			(justify left bottom)
 		)
 	)
